File: PortaPi_R1/PortaPi_R1.kicad_sch (KiCad schematic)
At the start: 59 parts, among them J1 Raspberry_Pi_2_3, J2 USB_C_Receptacle, J3 AudioJack3_Ground_Switch, J4 FPC 0.5mmP 18 Pin, SW1 SW_Push, SW2 SW_Slide_DPDT, U1 BQ24072RGT, U2 TPS61252DSG, U3 LTC2942, U4 BME680, U5 TPS7A0533PDBV, U6 CH340C, U7 RFM95W-915S2, U8 PCM5102A

Commit message: lots of new work and features
Parts:
- removed J3: AudioJack3_Ground_Switch, symbol Connector_Audio:AudioJack3_Ground_Switch
- removed SW1: SW_Push, symbol Switch:SW_Push
- removed U7: RFM95W-915S2, RF_Module:HOPERF_RFM9XW_SMD, symbol RF_Module:RFM95W-915S2
- removed U8: PCM5102A, Package_SO:TSSOP-20_4.4x6.5mm_P0.65mm, symbol Audio:PCM5102A
- added AE1: Antenna, RF_Antenna:Texas_SWRA416_868MHz_915MHz, symbol Device:Antenna
- added AE2: Antenna, RF_Antenna:Pulse_W3000, symbol Device:Antenna
- added C24: 100pF, Capacitor_SMD:C_0603_1608Metric, symbol Device:C
- added C25, C26, C27, C31, C35, C36, C44: 1uF, Capacitor_SMD:C_0805_2012Metric, symbol Device:C
- added C28, C29, C30, C45, C46, C47: 1uF, Capacitor_SMD:C_0603_1608Metric, symbol Device:C
- added C32, C49: 10uF, Capacitor_SMD:C_0805_2012Metric, symbol Device:C
- added C33, C34: ~, Capacitor_SMD:C_0805_2012Metric, symbol Device:C
- added C37, C38, C39, C40, C41: 100nF, Capacitor_SMD:C_0805_2012Metric, symbol Device:C
- added C42, C43: 220pf, Capacitor_SMD:C_0805_2012Metric, symbol Device:C
- added C48, C6, C64, C65, Cr2, Cr3, Cr4, Cr5, Cr6, Cr7: 100nF, Capacitor_SMD:C_0603_1608Metric, symbol Device:C
- added C50, C51: 27p, Capacitor_SMD:C_0402_1005Metric, symbol Device:C
- added C52, C53, C54, C56, C58, C59, C60, C61, C62, C63: 100n, Capacitor_SMD:C_0402_1005Metric, symbol Device:C
- added C55, C57: 1u, Capacitor_SMD:C_0402_1005Metric, symbol Device:C
- added C66: 120nF, Capacitor_SMD:C_0603_1608Metric, symbol Device:C
- added C67: 6.8nF, Capacitor_SMD:C_0603_1608Metric, symbol Device:C
- added FB2, FB3: FerriteBead_Small, symbol Device:FerriteBead_Small
- added J3: AudioJack4, symbol Connector_Audio:AudioJack4
- added J5: SpeakerOut, symbol Connector:Conn_01x02_Pin
- added J6: SIM_Card, symbol Connector:SIM_Card
- added J7: Conn_01x02, Connector_PinHeader_2.54mm:PinHeader_1x02_P2.54mm_Vertical, symbol Connector_Generic:Conn_01x02
- added L2: ~, Inductor_SMD:L_0805_2012Metric, symbol Device:L
- added R15, R16: 5.1k, Resistor_SMD:R_0603_1608Metric, symbol Device:R
- added R17, R19: 20k, Resistor_SMD:R_0603_1608Metric, symbol Device:R
- added R18: 1k, Resistor_SMD:R_0603_1608Metric, symbol Device:R
- added R20, R22: 1k, Capacitor_SMD:C_0402_1005Metric, symbol Device:R
- added R21: DNF, Capacitor_SMD:C_0402_1005Metric, symbol Device:R
- added R23, R24: 100k, Resistor_SMD:R_0603_1608Metric, symbol Device:R
- added TP1, TP2, TP3, TP4: TestPoint, symbol Connector:TestPoint
- added U10: W25Q128JVS, Package_SO:SOIC-8_5.23x5.23mm_P1.27mm, symbol RP2040_minimal-rescue:W25Q128JVS-Memory_Flash
- added U11: PAM8302AAD, symbol Amplifier_Audio:PAM8302AAD
- added U12, U14: TPS7A0533PDBV, Package_TO_SOT_SMD:SOT-23-5, symbol Regulator_Linear:TPS7A0533PDBV
- added U13: BG95M3LA-64-SGNS, BG95_QWS, symbol Quectel_BG95M3LA:BG95M3LA-64-SGNS
- added U15: RP2040, RP2040_minimal:RP2040-QFN-56, symbol MCU_RaspberryPi_RP2040:RP2040
- added U16: BNO055, Package_LGA:LGA-28_5.2x3.8mm_P0.5mm, symbol Sensor_Motion:BNO055
- added U7: RAK3172, RAK3172_RAK, symbol RAK3172:RAK3172
- added U8: TLV320AIC3101IRHBR, RHB32_3P45X3P45, symbol TI_TLV320AIC3101:TLV320AIC3101IRHBR
- added U9: PCAL6416AHF, Package_SO:SOIC-24W_7.5x15.4mm_P1.27mm, symbol Interface_Expansion:PCAL6416AHF
- added Y1: ABLS-12.000MHZ-B4-T, RP2040_minimal:Crystal_SMD_HC49-US, symbol Device:Crystal
- C10, C14, C15, C19, C20, C3, C4, C5: footprint (none) -> Capacitor_SMD:C_0805_2012Metric
- C11, C12, C13, C16, C17, C18, C2, C22, C23, C7, C8, C9: footprint (none) -> Capacitor_SMD:C_0603_1608Metric
- Cr1: renamed from C6; footprint (none) -> Capacitor_SMD:C_0603_1608Metric
- J2: footprint (none) -> Connector_USB:USB_C_Receptacle_GCT_USB4105-xx-A_16P_TopMnt_Horizontal
- R1, R10, R11, R2, R4, R5, R6, R7, R8, R9, TH1: footprint (none) -> Resistor_SMD:R_0603_1608Metric
Connections:
- net +3.3VA: now also C25.1, C26.1, C27.1, C32.1, C36.1, C44.1, C65.1, C66.1, C67.1, Cr2.1, Cr3.1, Cr4.1, Cr5.1, Cr7.1, J6.1 (VCC), R23.2, R24.2, U11.6 (VDD), U13.43 (USIM_VDD), U16.28 (VDDIO), U16.3 (VDD), U8.18 (DRVDD), U8.24 (DRVDD), U8.25 (AVDD), U8.7 (IOVDD), U9.21 (V_{DD(P)}), U9.23 (V_{DD(I2C-bus)})
- net +5V: now also C24.1, C28.1, C45.1, C6.1, U12.1 (IN), U14.1 (IN)
- net EYESPI_BUSY: now also U9.8 (P0_7)
- net EYESPI_CARDCS: now also U9.2 (P0_1)
- net EYESPI_GPIO1: now also U9.10 (P1_0)
- net EYESPI_GPIO2: now also U9.11 (P1_1)
- net EYESPI_INT: now also U9.7 (P0_6)
- net EYESPI_LITE: now also J1.33 (PWM1/GPIO13); no longer J1.32 (PWM0/GPIO12)
- net EYESPI_MEMCS: now also U9.3 (P0_2)
- net EYESPI_SCL: now also U16.19 (COM1), U8.8 (SCL), U9.19 (SCL)
- net EYESPI_SDA: now also U16.20 (COM0), U8.9 (SDA), U9.20 (SDA)
- net EYESPI_TFTCS: now also U9.1 (P0_0)
- net EYESPI_TFTDC: now also U9.5 (P0_4)
- net EYESPI_TFTRST: now also U9.6 (P0_5)
- net EYESPI_TSCS: now also U9.4 (P0_3)
- net GND: now also C24.2, C25.2, C26.2, C27.2, C28.2, C29.2, C30.2, C31.2, C32.2, C33.2, C34.2, C36.2, C42.1, C43.1, C44.2, C45.2, C46.2, C47.2, C48.2, C49.2, C50.2, C51.2, C52.2, C53.2, C54.2, C55.2, C56.2, C57.2, C58.2, C59.2, C6.2, C60.2, C61.2, C62.2, C63.2, C64.2, C65.2, C66.2, C67.2, Cr2.2, Cr3.2, Cr4.2, Cr5.2, Cr6.2, Cr7.2, J3.R2, J6.5 (GND), J7.2 (Pin_2), U10.4 (GND), U11.7 (GND), U12.2 (GND), U13.47 (USIM_GND), U14.2 (GND), U15.19 (TESTEN), U15.57 (GND), U16.15 (GNDIO), U16.16 (GNDIO), U16.17 (COM3), U16.18 (COM2), U16.2 (GND), U16.25 (GNDIO), U16.5 (PS1), U16.6 (PS0), U7.11 (GND), U7.17 (GND), U7.18 (GND), U7.23 (GND), U7.28 (GND), U8.17 (AVSS1), U8.21 (DRVSS), U8.26 (AVSS2), U8.33 (EPAD), U8.6 (DVSS), U9.18 (ADDR), U9.25 (EP), U9.9 (V_{SS})
- net I2S_BC: now also U8.2 (BCLK)
- net I2S_LRCLK: now also U8.3 (WCLK)
- net I2S_RXD: now also U8.5 (DOUT)
- net I2S_TXD: now also U8.4 (DIN)
- net at C3.1, SW2.2 (B), U1.10 (OUT)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: now also R15.2, R16.2; no longer D1.2 (A), D2.2 (A)
- net SWCLK: now reaches J1.13 (GPIO27)
- net SWCLK: now also U15.24 (SWCLK)
- net LoRaUART_TX: now reaches J1.15 (GPIO22)
- net LoRaUART_TX: now also U7.2 (PA2/UART2_TX)
- net LoRaUART_RX: now reaches J1.16 (GPIO23)
- net LoRaUART_RX: now also U7.1 (PA3/UART2_RX)
- net SWD: now reaches J1.37 (GPIO26)
- net SWD: now also U15.25 (SWD)
- net I2S_MCLK: now reaches J1.7 (GCLK0/GPIO4)
- net I2S_MCLK: now also U8.1 (MCLK)
- new net: R18.1, U8.15 (MICBIAS)
- new net: D2.2 (A), R16.1
- new net: C35.2, U8.16 (MIC2R/LINE2R)
- new net: C38.2, U8.19 (HPLOUT)
- new net: C37.2, U8.23 (HPROUT)
- new net: R19.2, U8.29 (RIGHT_LOP)
- new net: R17.2, U8.30 (RIGHT_LOM)
- new net: C51.1, R22.2, Y1.2
- new net: C64.1, U16.9 (CAP)
- new net: C34.1, L2.2, U7.12 (RF)
- new net: AE1.1 (A), C33.1, L2.1
- new net: D1.2 (A), R15.1
- new net: AE2.1 (A), U13.49 (ANT_GNSS)
- new net: TP1.1, U13.23 (DBG_TXD)
- new net: R24.1, U16.4 (~{BOOT_LOAD_PIN})
- new net: C40.1, U11.3 (IN+)
- new net: C39.1, C40.2, R17.1
- new net: TP3.1, U15.46 (USB_DM)
- new net: TP2.1, U15.47 (USB_DP)
- new net: C42.2, FB2.1, J5.2 (Pin_2)
- new net: TP4.1, U13.22 (DBG_RXD)
- new net: J6.2 (RST), U13.44 (USIM_RST)
- new net: J6.7 (I/O), U13.45 (USIM_DATA)
- new net: J6.3 (CLK), U13.46 (USIM_CLK)
- new net: C43.2, FB3.1, J5.1 (Pin_1)
- new net: C39.2, C41.2, R19.1
- new net: C41.1, U11.4 (IN-)
- new net: FB3.2, U11.5 (OUT+)
- new net: FB2.2, U11.8 (OUT-)
- new net +1V1: C53.1, C54.1, C55.1, U15.23 (DVDD), U15.45 (VREG_VOUT), U15.50 (DVDD)
- new net +1V8: C31.1, Cr6.1, U8.32 (DVDD)
- new net +3.3V_AUX1: C29.1, C30.1, C48.1, C49.1, U12.5 (OUT), U7.24 (VDD)
- new net +3.3V_AUX2: C46.1, C47.1, U13.29 (VDD_EXT), U14.5 (OUT)
- new net +3V3: C52.1, C56.1, C57.1, C58.1, C59.1, C60.1, C61.1, C62.1, C63.1, R21.1, U10.8 (VCC), U15.1 (IOVDD), U15.10 (IOVDD), U15.22 (IOVDD), U15.33 (IOVDD), U15.42 (IOVDD), U15.43 (ADC_AVDD), U15.44 (VREG_IN), U15.48 (USB_VDD), U15.49 (IOVDD)
- new net AudioAmp_SD: U11.1 (~{SD})
- new net CELL_RX: U13.34 (MAIN_RXD)
- new net CELL_TX: U13.35 (MAIN_TXD)
- new net EN_3.3Aux1: U12.3 (EN)
- new net EN_3.3Aux2: U14.3 (EN)
- new net EXPANDER_INT: U9.22 (~{INT})
- new net HP_L: C38.1, J3.T
- new net HP_MIC: C35.1, J3.S, R18.2, U8.14 (MIC2L/LINE2L/MICDET)
- new net HP_R: C37.1, J3.R1
- new net QSPI_SCLK: U10.6 (CLK), U15.52 (QSPI_SCLK)
- new net QSPI_SD0: U10.5 (DI(IO0)), U15.53 (QSPI_SD0)
- new net QSPI_SD1: U10.2 (DO(IO1)), U15.55 (QSPI_SD1)
- new net QSPI_SD2: U10.3 (IO2), U15.54 (QSPI_SD2)
- new net QSPI_SD3: U10.7 (IO3), U15.51 (QSPI_SD3)
- new net QSPI_SS: R20.1, R21.2, U10.1 (~{CS}), U15.56 (QSPI_SS)
- new net RESET: R23.1, U13.17 (RESET_N), U16.11 (~{RESET}), U7.22 (RST), U8.31 (*RESET), U9.24 (~{RESET})
- new net RUN: U15.26 (RUN)
- new net XIN: C50.1, U15.20 (XIN), Y1.1
- new net XOUT: R22.1, U15.21 (XOUT)
- new net ~{USB_BOOT}: J7.1 (Pin_1), R20.2
Other:
- note added: "6.6 V Input OVP Battery Short Circuit Protection NTC Temperature shutdown"
- note added: "7bit I2C Address = 0x32"
- note added: "Audio Codec"
- note added: "Audio I2S"
- note added: "Audio Jack"
- note added: "Buck/Boost"
- note added: "Built-In Mono Speaker"
- note added: "Cell Module"
- note added: "Coulomb Counter"
- note added: "Crystal"
- note added: "Display SPI0"
- note added: "Headphones"
- note added: "I/O Expander for system use."
- note added: "IMU"
- note added: "LDO"
- note added: "LoRa SW Serial"
- note added: "Make sure C10 is close to pin 44 of RP2040"
- note added: "Make sure C8 is close to pin 45 of RP2040"
- note added: "No PD USB 2.0"
- note added: "ON/OFF"
- note added: "PWM0"
- note added: "Power Path/Charging"
- note added: "RP2040"
- note added: "RP2040 Flash"
- note added: "RP2040 Prog"
- note added: "RasPi Header"
- note added: "Speaker"
- note added: "Sys I2C Bus"
- note added: "Temperature/Pressure Sensor"
- note added: "USB C"
- note added: "USB UART0"
- note added: "USB/UART"
- note removed: "Battery Power Path/Charging IC 6.6 V Input OVP Battery Short Circuit Protection NTC Temperature shutdown"
- note removed: "Temperature/Pressure/Environment Sensor"
- note removed: "USB C No PD USB 2.0"
- note removed: "todo: interface the CS stuff so that we can really rip these screens"
- title: (none) -> PortaPi BackPack Board 
- moved on the sheet: BT1, C1, C10, C11, C12, C13, C14, C15, C16, C17, C18, C19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

Commit message: starting layout
Parts:
- removed C21: 100nF, symbol Device:C
- removed TP2, TP3: TestPoint, symbol Connector:TestPoint
- removed U6: CH340C, Package_SO:SOIC-16_3.9x9.9mm_P1.27mm, symbol Interface_USB:CH340C
- removed U9: PCAL6416AHF, Package_SO:SOIC-24W_7.5x15.4mm_P1.27mm, symbol Interface_Expansion:PCAL6416AHF
- added H1, H2, H3, H4: MountingHole_Pad, MountingHole:MountingHole_2.5mm_Pad_Via, symbol Mechanical:MountingHole_Pad
- added J8, J9: DF40HC3.0-30DS-0.4V51, CONN_30DS-0.4V51, symbol DF40HC:DF40HC3.0-30DS-0.4V51
- added R25, R26, R27, R28, R29, R30: 22, Capacitor_SMD:C_0402_1005Metric, symbol Device:R
- J1: footprint Connector_PinSocket_2.54mm:PinSocket_2x20_P2.54mm_Vertical -> Module:Raspberry_Pi_Zero_Socketed_THT_FaceDown_MountingHoles
- U13: footprint BG95_QWS -> Quectel_BG95M3LA:BG95_QWS
- U15: footprint RP2040_minimal:RP2040-QFN-56 -> Package_DFN_QFN:QFN-56-1EP_7x7mm_P0.4mm_EP3.2x3.2mm
Connections:
- net EYESPI_BUSY: now also U15.34 (GPIO22)
- net EYESPI_CARDCS: now also U15.27 (GPIO16)
- net EYESPI_GPIO1: now also U15.36 (GPIO24)
- net EYESPI_GPIO2: now also U15.37 (GPIO25)
- net EYESPI_INT: now also U15.32 (GPIO21)
- net EYESPI_MEMCS: now also U15.28 (GPIO17)
- net EYESPI_SCL: now also U15.12 (GPIO9)
- net EYESPI_SDA: now also U15.11 (GPIO8)
- net EYESPI_TFTCS: now also U15.18 (GPIO15)
- net EYESPI_TFTDC: now also U15.30 (GPIO19)
- net EYESPI_TFTRST: now also U15.31 (GPIO20)
- net EYESPI_TSCS: now also U15.29 (GPIO18)
- net GND: now also H1.1, H2.1, H3.1, H4.1
- net LoRaUART_RX: now also R29.1; no longer J1.16 (GPIO23)
- net LoRaUART_TX: now also R30.1; no longer J1.15 (GPIO22)
- net UART0_RXD: now also R25.1
- net UART0_TXD: now also R26.1
- net USB_DM: now reaches D3.1 (K), J2.A7 (D-), J2.B7 (D-)
- net USB_DM: now also R28.1
- net USB_DP: now reaches D3.3 (K), J2.A6 (D+), J2.B6 (D+)
- net USB_DP: now also R27.1
- net at U15.46 (USB_DM): now also R28.2
- net at U15.47 (USB_DP): now also R27.2
- net at U15.2 (GPIO0): now also R25.2
- net at U15.3 (GPIO1): now also R26.2
- net at U15.6 (GPIO4): now also R29.2
- net at U15.7 (GPIO5): now also R30.2
Other:
- note added: "GPIO Expansion"
- note added: "LoRa UART1"
- note added: "RP2040 UART0"
- note added: "RPi Uart 0"
- note added: "USB"
- note removed: "7bit I2C Address = 0x32"
- note removed: "I/O Expander for system use."
- note removed: "LoRa SW Serial"
- note removed: "USB UART0"

Commit message: placing and routing
Parts:
- removed C11: 100pF, Capacitor_SMD:C_0603_1608Metric, symbol Device:C
- removed C4: 10uF, Capacitor_SMD:C_0805_2012Metric, symbol Device:C
- removed Cr1: 100nF, Capacitor_SMD:C_0603_1608Metric, symbol Device:C
- added SW1, SW3, SW4, SW5: SW_SPST, Button_Switch_THT:SW_Tactile_SPST_Angled_PTS645Vx31-2LFS, symbol Switch:SW_SPST
- BT1: footprint (none) -> Connector_JST:JST_PH_S2B-PH-SM4-TB_1x02-1MP_P2.00mm_Horizontal
- C1: footprint (none) -> Capacitor_SMD:C_0805_2012Metric
- C50, C51: value 27p -> 27pf
- D1, D2: footprint (none) -> LED_SMD:LED_0603_1608Metric
- F1, FB1, R3: footprint (none) -> Resistor_SMD:R_0603_1608Metric
- L1: footprint (none) -> Inductor_SMD:L_Bourns-SRN4018
- SW2: footprint (none) -> Button_Switch_SMD:SW_SPDT_PCM12
- Y1: value ABLS-12.000MHZ-B4-T -> ABM3-12.000MHZ-D2Y-T; footprint RP2040_minimal:Crystal_SMD_HC49-US -> Crystal:Crystal_SMD_5032-4Pin_5.0x3.2mm
Other:
- note added: "L and R bumpers?"

Commit message: routing work
Parts:
- added C11, C4: 220pf, Capacitor_SMD:C_0805_2012Metric, symbol Device:C
- added C21: 1uF, Capacitor_SMD:C_0805_2012Metric, symbol Device:C
- added C68, C69, C70: 100nF, Capacitor_SMD:C_0805_2012Metric, symbol Device:C
- added Cr1: 100nF, Capacitor_SMD:C_0603_1608Metric, symbol Device:C
- added D4: ESDA5V3SC5, Package_TO_SOT_SMD:SOT-23-5, symbol Power_Protection:ESDA5V3SC5
- added FB4, FB5: FerriteBead_Small, symbol Device:FerriteBead_Small
- added J10: SpeakerOut, symbol Connector:Conn_01x02_Pin
- added R31: 20k, Resistor_SMD:R_0603_1608Metric, symbol Device:R
- added SW10, SW11, SW12, SW13, SW14, SW15, SW6, SW7, SW8, SW9: SW_SPST, Button_Switch_SMD:SW_SPST_SKQG_WithoutStem, symbol Switch:SW_SPST
- added U6: PAM8302AAD, Package_SO:SOP-8_3.9x4.9mm_P1.27mm, symbol Amplifier_Audio:PAM8302AAD
- C52: footprint Capacitor_SMD:C_0402_1005Metric -> Capacitor_SMD:C_0603_1608Metric
- U11: footprint (none) -> Package_SO:SOP-8_3.9x4.9mm_P1.27mm
Connections:
- net AudioAmp_SD: now also U6.1 (~{SD})
- net GND: now also C21.2, Cr1.2, D4.2 (A), U6.7 (GND)
- net HP_L: now also D4.1 (K)
- net HP_MIC: now also D4.4 (K)
- net HP_R: now also D4.3 (K)
- new net: C4.2, FB4.1, J10.1 (Pin_1)
- new net: C11.2, FB5.1, J10.2 (Pin_2)
- new net: C69.1, U6.4 (IN-)
- new net: C69.2, C70.2, R31.1
- new net: FB4.2, U6.5 (OUT+)
- new net: C68.2, C70.1
- new net: C68.1, U6.3 (IN+)
- new net: C21.1, Cr1.1, U6.6 (VDD)
- new net: FB5.2, U6.8 (OUT-)
Other:
- moved on the sheet: D3

Commit message: lots more routing work
Parts:
- removed AE1: Antenna, RF_Antenna:Texas_SWRA416_868MHz_915MHz, symbol Device:Antenna
- removed AE2: Antenna, RF_Antenna:Pulse_W3000, symbol Device:Antenna
- added J11, J12: DF40HC3.0-30DP, DF40C-30DP:SOIC_0DP-0.4V51_HIR, symbol DF40HC:DF40HC3.0-30DS-0.4V51
- added J13, J14: Conn_Coaxial_Small, Connector_Coaxial:U.FL_Molex_MCRF_73412-0110_Vertical, symbol Connector:Conn_Coaxial_Small
- added R32, R33, R34, R35, R36, R37, R38, R39, R40, R41, R42, R43, R44, R45, R46: 20k, Resistor_SMD:R_0603_1608Metric, symbol Device:R
- added U9: PCAL6416AHF, Package_DFN_QFN:HVQFN-24-1EP_4x4mm_P0.5mm_EP2.1x2.1mm, symbol Interface_Expansion:PCAL6416AHF
- C35, C37, C38, C39, C40, C41: footprint Capacitor_SMD:C_0805_2012Metric -> Capacitor_SMD:C_0603_1608Metric
- R18: footprint Resistor_SMD:R_0603_1608Metric -> Capacitor_SMD:C_0603_1608Metric
- SW10: value SW_SPST -> L; footprint Button_Switch_SMD:SW_SPST_SKQG_WithoutStem -> Button_Switch_THT:SW_PUSH_6mm
- SW11: value SW_SPST -> R; footprint Button_Switch_SMD:SW_SPST_SKQG_WithoutStem -> Button_Switch_THT:SW_PUSH_6mm
- SW12: value SW_SPST -> U; footprint Button_Switch_SMD:SW_SPST_SKQG_WithoutStem -> Button_Switch_THT:SW_PUSH_6mm
- SW13: value SW_SPST -> D; footprint Button_Switch_SMD:SW_SPST_SKQG_WithoutStem -> Button_Switch_THT:SW_PUSH_6mm
- SW14, SW15: footprint Button_Switch_SMD:SW_SPST_SKQG_WithoutStem -> Button_Switch_THT:SW_PUSH_6mm
- SW6: value SW_SPST -> A; footprint Button_Switch_SMD:SW_SPST_SKQG_WithoutStem -> Button_Switch_THT:SW_PUSH_6mm
- SW7: value SW_SPST -> X; footprint Button_Switch_SMD:SW_SPST_SKQG_WithoutStem -> Button_Switch_THT:SW_PUSH_6mm
- SW8: value SW_SPST -> B; footprint Button_Switch_SMD:SW_SPST_SKQG_WithoutStem -> Button_Switch_THT:SW_PUSH_6mm
- SW9: value SW_SPST -> Y; footprint Button_Switch_SMD:SW_SPST_SKQG_WithoutStem -> Button_Switch_THT:SW_PUSH_6mm
Connections:
- net +3.3V: now also R33.2, R34.2, R35.2, R36.2, R37.2, R38.2, R39.2, R40.2, R41.2, R42.2, R43.2, R44.2, R45.2, R46.2
- net +3.3VA: now also C21.1, Cr1.1, J8.19, J9.12, U11.1 (~{SD}), U6.6 (VDD)
- net +3.3V_AUX1: now also J8.4, J9.27
- net EYESPI_SCL: now also J8.15, J9.1, U13.40 (I2C_SCL), U7.9 (PA12/I2C_SCL), U9.19 (SCL)
- net EYESPI_SDA: now also J8.30, J9.16, U13.41 (I2C_SDA), U7.10 (PA11/I2C_SDA), U9.20 (SDA)
- net GND: now also C11.1, C4.1, J8.14, J8.17, J8.2, J8.29, J9.14, J9.17, J9.2, J9.29, SW1.2 (B), SW10.2 (B), SW11.2 (B), SW12.2 (B), SW13.2 (B), SW14.2 (B), SW15.2 (B), SW3.2 (B), SW4.2 (B), SW5.2 (B), SW6.2 (B), SW7.2 (B), SW8.2 (B), SW9.2 (B), U13.3 (GND), U13.31 (GND), U13.48 (GND), U13.50 (GND), J13.2 (Ext), J14.2 (Ext), U9.18 (ADDR), U9.25 (EP), U9.9 (V_{SS})
- net RESET: now also U9.24 (~{RESET})
- net at U8.27 (LEFT_LOP): now also R19.2
- net at U8.28 (LEFT_LOM): now also R17.2
- net at U8.29 (RIGHT_LOP): now also R31.2; no longer R19.2
- net at U8.30 (RIGHT_LOM): now also R32.2; no longer R17.2
- net at C33.1, L2.1: now also J13.1 (In)
- net at U13.49 (ANT_GNSS): now also J14.1 (In)
- net RIGHT_LOP: now reaches U6.4 (IN-)
- net RIGHT_LOP: no longer C69.1
- net BUTTON_D: now reaches SW13.1 (A)
- net BUTTON_D: now also R40.1, U9.8 (P0_7)
- net LEFT_LOM: now reaches U11.3 (IN+)
- net LEFT_LOM: no longer C40.1
- net BUTTON_U: now reaches SW12.1 (A)
- net BUTTON_U: now also R36.1, U9.7 (P0_6)
- net at C42.2, FB2.1: now also J5.1 (Pin_1); no longer J5.2 (Pin_2)
- net BUTTON_L2: now reaches SW1.1 (A)
- net BUTTON_L2: now also U15.9 (GPIO7), R46.1
- net BUTTON_Y: now reaches SW9.1 (A)
- net BUTTON_Y: now also R38.1, U9.4 (P0_3)
- net at C68.2, C70.1: now also R32.1
- net LEFT_LOP_CON: now reaches J8.13
- net LEFT_LOP_CON: now also C41.1
- net RIGHT_LOM_CON: now reaches J8.18
- net RIGHT_LOM_CON: now also C68.1
- net LEFT_LOM_CON: now reaches J8.28
- net LEFT_LOM_CON: now also C40.1
- net RIGHT_LOP_CON: now reaches J8.3
- net RIGHT_LOP_CON: now also C69.1
- net BUTTON_X: now reaches SW7.1 (A)
- net BUTTON_X: now also R37.1, U9.3 (P0_2)
- net BUTTON_R1: now reaches SW4.1 (A)
- net BUTTON_R1: now also U15.13 (GPIO10), R45.1
- net RIGHT_LOM: now reaches U6.3 (IN+)
- net RIGHT_LOM: no longer C68.1
- net at C43.2, FB3.1: now also J5.2 (Pin_2); no longer J5.1 (Pin_1)
- net BUTTON_R: now reaches SW11.1 (A)
- net BUTTON_R: now also R39.1, U9.6 (P0_5)
- net BUTTON_L: now reaches SW10.1 (A)
- net BUTTON_L: now also R35.1, U9.5 (P0_4)
- net BUTTON_R2: now reaches SW5.1 (A)
- net BUTTON_R2: now also U15.14 (GPIO11), R44.1
- net BUTTON_L1: now reaches SW3.1 (A)
- net BUTTON_L1: now also U15.8 (GPIO6), R43.1
- net BUTTON_START: now reaches SW14.1 (A)
- net BUTTON_START: now also R41.1, U9.10 (P1_0)
- net LEFT_LOP: now reaches U11.4 (IN-)
- net LEFT_LOP: no longer C41.1
- net at U11.5 (OUT+): now also FB2.2; no longer FB3.2
- net at U11.8 (OUT-): now also FB3.2; no longer FB2.2
- net BUTTON_B: now reaches SW8.1 (A)
- net BUTTON_B: now also R34.1, U9.2 (P0_1)
- net BUTTON_SELECT: now reaches SW15.1 (A)
- net BUTTON_SELECT: now also R42.1, U9.11 (P1_1)
- net BUTTON_A: now reaches SW6.1 (A)
- net BUTTON_A: now also R33.1, U9.1 (P0_0)
- net AudioAmp_SD: no longer names the net of U6.1 (~{SD})
- net AudioAmp_SD: no longer U11.1 (~{SD})
Other:
- note added: "Built-In Left Speaker"
- note added: "Built-In Right Speaker"
- note removed: "Built-In Mono Speaker"
- moved on the sheet: C39, C40, C41, C50, C51, J6, J7, J8, J9, R17, R19, R22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
