File: PortaPi_R1/PortaPi_R1.kicad_sch (KiCad schematic)
At the start: 189 parts, among them J1 Raspberry_Pi_2_3, J10 SpeakerOut, J11 DF40HC3.0-30DP, J12 DF40HC3.0-30DP, J13 Conn_Coaxial_Small, J14 Conn_Coaxial_Small, J2 USB_C_Receptacle, J3 AudioJack4, J4 FPC 0.5mmP 18 Pin, J5 SpeakerOut, J6 SIM_Card, J7 Conn_01x02, J8 DF40HC3.0-30DS-0.4V51, J9 DF40HC3.0-30DS-0.4V51, SW1 SW_SPST, SW10 L, SW11 R, SW12 U, SW13 D, SW14 SW_SPST, SW15 SW_SPST, SW2 SW_Slide_DPDT, SW3 SW_SPST, SW4 SW_SPST, SW5 SW_SPST, SW6 A, SW7 X, SW8 B, SW9 Y, U1 BQ24072RGT, U10 W25Q128JVS, U11 PAM8302AAD, U12 TPS7A0533PDBV, U13 BG95M3LA-64-SGNS, U14 TPS7A0533PDBV, U15 RP2040, U16 BNO055, U2 TPS61252DSG, U3 LTC2942, U4 BME680, U5 TPS7A0533PDBV, U6 PAM8302AAD, U7 RAK3172, U8 TLV320AIC3101IRHBR, U9 PCAL6416AHF, Y1 ABM3-12.000MHZ-D2Y-T

Commit message: placing work
Parts:
- removed C33, C34: ~, Capacitor_SMD:C_0805_2012Metric, symbol Device:C
- removed J6: SIM_Card, symbol Connector:SIM_Card
- removed J7: Conn_01x02, Connector_PinHeader_2.54mm:PinHeader_1x02_P2.54mm_Vertical, symbol Connector_Generic:Conn_01x02
- removed L2: ~, Inductor_SMD:L_0805_2012Metric, symbol Device:L
- removed R12: 0, symbol Device:R
- added D5, D6, D7, D8: WS2812, LED_SMD:LED_WS2812_PLCC6_5.0x5.0mm_P1.6mm, symbol LED:WS2812
- added SW12: BOOT, Button_Switch_SMD:SW_SPST_B3U-1000P-B, symbol Switch:SW_SPST
- added U13: SM351LT, Package_TO_SOT_SMD:SOT-23, symbol Sensor_Magnetic:SM351LT
- added U16: 1042240820, 1042240820:1042240820_MOL, symbol 1042240820:1042240820
- C27: renamed from C36; footprint Capacitor_SMD:C_0805_2012Metric -> Capacitor_SMD:C_0603_1608Metric
- C29: renamed from C25; footprint Capacitor_SMD:C_0805_2012Metric -> Capacitor_SMD:C_0603_1608Metric
- C31: renamed from C68; footprint Capacitor_SMD:C_0805_2012Metric -> Capacitor_SMD:C_0603_1608Metric
- C32: renamed from C70; footprint Capacitor_SMD:C_0805_2012Metric -> Capacitor_SMD:C_0603_1608Metric
- C33: renamed from C69; footprint Capacitor_SMD:C_0805_2012Metric -> Capacitor_SMD:C_0603_1608Metric
- C35: renamed from C31; footprint Capacitor_SMD:C_0805_2012Metric -> Capacitor_SMD:C_0603_1608Metric
- C37: renamed from C26; footprint Capacitor_SMD:C_0805_2012Metric -> Capacitor_SMD:C_0603_1608Metric
- C39: renamed from C27; footprint Capacitor_SMD:C_0805_2012Metric -> Capacitor_SMD:C_0603_1608Metric
- C53: renamed from C48; now not fitted
- C54: renamed from C49; now not fitted
- FB2: renamed from FB4; footprint (none) -> Inductor_SMD:L_0603_1608Metric
- FB3: renamed from FB5; footprint (none) -> Inductor_SMD:L_0603_1608Metric
- FB4: renamed from FB2; footprint (none) -> Inductor_SMD:L_0603_1608Metric
- FB5: renamed from FB3; footprint (none) -> Inductor_SMD:L_0603_1608Metric
- J11: renamed from J13; now not fitted
- J12: renamed from J14; now not fitted
- J2: renamed from J9; footprint CONN_30DS-0.4V51 -> DF40HC:CONN_30DS-0.4V51
- J7: renamed from J3; footprint (none) -> Connector_Audio:Jack_3.5mm_PJ320D_Horizontal
- J8: footprint CONN_30DS-0.4V51 -> DF40HC:CONN_30DS-0.4V51
- R30: renamed from R13; footprint (none) -> Resistor_SMD:R_0603_1608Metric
- R31: renamed from R14; footprint (none) -> Resistor_SMD:R_0603_1608Metric
- U12: renamed from U7; footprint RAK3172_RAK -> RAK3172:RAK3172_RAK
- U9: renamed from U8; footprint RHB32_3P45X3P45 -> TI_TLV320AIC3101:RHB32_3P45X3P45
- renumbered C3 to C1, C13 to C10, C9 to C11, C10 to C12, C14 to C13, C15 to C14, C28 to C15, C29 to C16, C30 to C17, C8 to C18, C45 to C19, C46 to C20, C47 to C21, C24 to C22, C6 to C23, C20 to C24, C19 to C25, Cr2 to C26, Cr3 to C28, C16 to C3, C32 to C30, Cr6 to C34, Cr4 to C36, Cr5 to C38, C17 to C4, C21 to C40, C4 to C41, C40 to C42, C11 to C43, C39 to C44, C41 to C45, C38 to C46, C37 to C47, C35 to C48, C44 to C49, C18 to C5, Cr7 to C50, C42 to C51, C43 to C52, C22 to C55, C23 to C56, C53 to C57, C54 to C58, C56 to C59, C7 to C6, C58 to C60, C59 to C61, C60 to C62, C61 to C63, C62 to C64, C63 to C65, C55 to C66, C57 to C67, C52 to C68, C65 to C69, C12 to C7, C66 to C70, C67 to C71, C50 to C72, C51 to C73, C64 to C74, Cr1 to C75, C5 to C8, C1 to C9, J2 to J1, J5 to J10, J12 to J3, J1 to J5, J10 to J6, J11 to J9, R3 to R1, R15 to R10, R10 to R11, R33 to R12, R37 to R13, R23 to R14, R34 to R15, R38 to R16, R35 to R17, R39 to R18, R36 to R19, R6 to R2, R40 to R20, R41 to R21, R42 to R22, R32 to R23, R31 to R24, R4 to R25, R5 to R26, R17 to R27, R19 to R28, R18 to R29, R7 to R3, R27 to R32, R28 to R33, R25 to R34, R26 to R35, R21 to R36, R29 to R37, R30 to R38, R20 to R39, R1 to R4, R24 to R40, R22 to R41, R46 to R42, R45 to R44, R44 to R45, R2 to R5, R11 to R6, R9 to R7, R16 to R8, R8 to R9, SW2 to SW1, SW14 to SW10, SW15 to SW11, SW1 to SW13, SW3 to SW14, SW4 to SW15, SW5 to SW16, SW6 to SW2, SW7 to SW3, SW8 to SW4, SW9 to SW5, SW10 to SW6, SW11 to SW7, SW12 to SW8, SW13 to SW9, TP4 to TP1, TP1 to TP2, U5 to U1, U11 to U10, U4 to U11, U10 to U14, U16 to U17, U13 to U18, U1 to U2, U2 to U3, U12 to U4, U3 to U5, U14 to U6, U9 to U7, U6 to U8
Connections:
- net +3.3V: now also J2.12, J2.19, J8.12, J8.19
- net +3.3VA: now also U16.S1 (VCC); no longer J2.12, J8.19
- net +3.3V_AUX1: now also J2.4, J8.27
- net +5V: now also J2.23, J2.8, J3.23, J3.8, J8.23, J8.8, J9.8
- net EYESPI_SCL: now also J2.15, J8.16, J9.15
- net EYESPI_SDA: now also J2.30, J8.1, J9.30
- net GND: now also J3.14, J3.17, J3.2, J3.29, J9.14, J9.17, J9.2, J9.29, D5.6 (VSS), D6.6 (VSS), D7.6 (VSS), D8.6 (VSS), SW12.1 (A), U16.G1 (GND), U16.G2 (GND), U16.G3 (GND), U16.G4 (GND), U16.S4 (GND)
- net LEFT_LOM: now also J9.28
- net LEFT_LOP: now also J9.13
- net RIGHT_LOM: now also J9.18
- net RIGHT_LOP: now also J9.3
- net ~{USB_BOOT}: now also SW12.2 (B)
- net at U12.12 (RF): now also J11.1 (In)
- net at U18.44 (USIM_RST): now also U16.S2 (RST)
- net at U18.45 (USIM_DATA): now also U16.S6 (I/O)
- net at U18.46 (USIM_CLK): now also U16.S3 (CLK)
- new net: D6.1 (DOUT), D7.2 (DIN)
- new net: D5.1 (DOUT), D6.2 (DIN)
- new net: D7.1 (DOUT), D8.2 (DIN)
Other:
- moved on the sheet: BT1, C1, C10, C11, C12, C13, C14, C15, C16, C17, C18, C19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

Commit message: routing and placinggit add .!
Parts:
- removed D5, D6, D7, D8: WS2812, LED_SMD:LED_WS2812_PLCC6_5.0x5.0mm_P1.6mm, symbol LED:WS2812
- added C76, C77: 100n, Capacitor_SMD:C_0402_1005Metric, symbol Device:C
- added D5, D6, D7, D9: WS2812B, LED_SMD:LED_WS2812B_PLCC4_5.0x5.0mm_P3.2mm, symbol LED:WS2812B
- added FID1, FID2, FID3, FID4: Fiducial, Fiducial:Fiducial_1.5mm_Mask3mm, symbol Mechanical:Fiducial
- C40, C41, C43, C49, C51, C52: footprint Capacitor_SMD:C_0805_2012Metric -> Capacitor_SMD:C_0603_1608Metric
- J10, J6: footprint (none) -> Jumper:SolderJumper-2_P1.3mm_Open_Pad1.0x1.5mm
Connections:
- net +3.3V: now also U7.21 (V_{DD(P)}), U7.23 (V_{DD(I2C-bus)}), C76.1, C77.1; no longer J5.1 (3V3), J5.17 (3V3)
- net +3.3VA: no longer C4.1, C5.1, U1.5 (OUT)
- net +3V3: now also C4.1, C5.1, U1.5 (OUT)
- net +5V: now also D5.1 (VDD), D6.1 (VDD), D7.1 (VDD), D9.1 (VDD)
- net EYESPI_LITE: now also U15.35 (GPIO23); no longer J5.33 (PWM1/GPIO13)
- net GND: now also C76.2, C77.2, D5.3 (VSS), D6.3 (VSS), D7.3 (VSS), D9.3 (VSS)
- net XIN: now also Y1.2; no longer Y1.1
- net at C73.1, R41.2: now also Y1.1; no longer Y1.2
- new net: D6.2 (DOUT), D7.4 (DIN)
- new net: D5.2 (DOUT), D6.4 (DIN)
- new net: D5.4 (DIN), D9.2 (DOUT)
- new net: J5.1 (3V3), J5.17 (3V3)
Other:
- note added: "Space for 20mm speaker"
- moved on the sheet: H1, H2, H3, H4, Y1

Commit message: routing...
Parts:
- added FID5, FID6, FID7, FID8: Fiducial, Fiducial:Fiducial_1.5mm_Mask3mm, symbol Mechanical:Fiducial
Connections:
- net +3.3V: now also R14.2
- net +3.3VA: no longer C26.1, C27.1, C28.1, C29.1, C30.1, C36.1, C37.1, C38.1, C39.1, C40.1, C49.1, C50.1, C55.1, C56.1, C69.1, C70.1, C71.1, C75.1, R14.2, R30.2, U10.6 (VDD), U11.6 (VDDIO), U11.8 (VDD), U17.28 (VDDIO), U17.3 (VDD), U8.6 (VDD), U9.18 (DRVDD), U9.24 (DRVDD), U9.25 (AVDD), U9.7 (IOVDD)
- net +3.3V_AUX1: now also C55.1, C56.1, C69.1, C70.1, C71.1, R30.2, U11.6 (VDDIO), U11.8 (VDD), U17.28 (VDDIO), U17.3 (VDD)
- net +3.3V_AUX2: now also C26.1, C27.1, C28.1, C29.1, C30.1, C36.1, C37.1, C38.1, C39.1, C40.1, C49.1, C50.1, C75.1, U10.6 (VDD), U8.6 (VDD), U9.18 (DRVDD), U9.24 (DRVDD), U9.25 (AVDD), U9.7 (IOVDD)
Other:
- moved on the sheet: FID1, FID2, FID3, FID4, R14

Commit message: routing
Parts:
- added C78, C79, C80: 1uF, Capacitor_SMD:C_0603_1608Metric, symbol Device:C
- added U19: TPS7A0533PDBV, Package_TO_SOT_SMD:SOT-23-5, symbol Regulator_Linear:TPS7A0533PDBV
Connections:
- net +3.3V: no longer C76.1, C77.1, R12.2, R13.2, R15.2, R16.2, R17.2, R18.2, R19.2, R20.2, R21.2, R22.2, U7.21 (V_{DD(P)}), U7.23 (V_{DD(I2C-bus)})
- net +3.3V_AUX1: now also R40.2; no longer C55.1, C56.1, J2.27, J2.4, J8.27, J8.4, R30.2, U11.6 (VDDIO), U11.8 (VDD)
- net +3.3V_AUX2: now also J2.27, J2.4, J4.1 (Pin_1), J8.27, J8.4; no longer C40.1, C49.1, C50.1, C75.1, U10.6 (VDD), U18.29 (VDD_EXT), U8.6 (VDD)
- net +3V3: now also C55.1, C56.1, R30.2, U11.6 (VDDIO), U11.8 (VDD)
- net +5V: now also C78.1, U19.1 (IN); no longer D5.1 (VDD), D6.1 (VDD), D7.1 (VDD), D9.1 (VDD), J3.23, J3.8, J9.8
- net EYESPI_SCL: no longer J9.15, U7.19 (SCL)
- net EYESPI_SDA: no longer J9.30, U7.20 (SDA)
- net GND: now also C78.2, C79.2, C80.2, U19.2 (GND); no longer C40.2, C41.1, C43.1, C49.2, C50.2, C51.1, C52.1, C75.2, C76.2, C77.2, D5.3 (VSS), D6.3 (VSS), D7.3 (VSS), D9.3 (VSS), J3.14, J3.17, J3.2, J3.29, J9.14, J9.17, J9.2, J9.29, SW10.2 (B), SW11.2 (B), SW2.2 (B), SW3.2 (B), SW4.2 (B), SW5.2 (B), SW6.2 (B), SW7.2 (B), SW8.2 (B), SW9.2 (B), U10.7 (GND), U7.18 (ADDR), U7.25 (EP), U7.9 (V_{SS}), U8.7 (GND)
- net I2C1_SCL_C: now reaches J3.1
- net I2C1_SCL_C: now also J3.15, J9.15, J9.16, U7.19 (SCL)
- net +3.3V_C: now reaches J3.12
- net +3.3V_C: now also C76.1, C77.1, J3.19, J9.12, J9.19, R12.2, R13.2, R15.2, R16.2, R17.2, R18.2, R19.2, R20.2, R21.2, R22.2, U7.21 (V_{DD(P)}), U7.23 (V_{DD(I2C-bus)})
- net I2C1_SDA_C: now reaches J3.16
- net I2C1_SDA_C: now also J3.30, J9.1, J9.30, U7.20 (SDA)
- net +3.3V_AUX2_C: now reaches J3.27
- net +3.3V_AUX2_C: now also C40.1, C49.1, C50.1, C75.1, J3.4, J9.27, J9.4, U10.6 (VDD), U8.6 (VDD)
- net +5V_C: now reaches J9.23
- net +5V_C: now also D5.1 (VDD), D6.1 (VDD), D7.1 (VDD), D9.1 (VDD), J3.23, J3.8, J9.8
- net INPUT_INT: now reaches U7.22 (~{INT})
- net GND_C: now reaches U8.1 (~{SD})
- net GND_C: now also C40.2, C41.1, C43.1, C49.2, C50.2, C51.1, C52.1, C75.2, C76.2, C77.2, D5.3 (VSS), D6.3 (VSS), D7.3 (VSS), D9.3 (VSS), J3.14, J3.17, J3.2, J3.29, J9.14, J9.17, J9.2, J9.29, SW10.2 (B), SW11.2 (B), SW2.2 (B), SW3.2 (B), SW4.2 (B), SW5.2 (B), SW6.2 (B), SW7.2 (B), SW8.2 (B), SW9.2 (B), U10.1 (~{SD}), U10.7 (GND), U7.18 (ADDR), U7.25 (EP), U7.9 (V_{SS}), U8.7 (GND)
- removed net +3.3VA: J4.1 (Pin_1), R40.2, U10.1 (~{SD}), U16.S1 (VCC), U18.43 (USIM_VDD)
- net LEFT_LOM renamed LEFT_LOM_C
- net LEFT_LOP renamed LEFT_LOP_C
- net RIGHT_LOM renamed RIGHT_LOM_C
- net RIGHT_LOP renamed RIGHT_LOP_C
- new net +3.3V_CELL: C79.1, C80.1, U16.S1 (VCC), U18.29 (VDD_EXT), U18.43 (USIM_VDD), U19.5 (OUT)
Other:
- note added: "Cell Radio"
- note added: "Cell Radio Audio Codec Speaker Display Vin"
- note added: "IMU LoRa Radio"
- note added: "RP2040 TempPresure Sensor Pull-Ups"
- note added: "i2c bus"
- moved on the sheet: C40, C41, C43, C49, C50, C51, C52, C75, FB2, FB3, FB4, FB5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

Commit message: nearly done routing....
Parts:
- removed J12: Conn_Coaxial_Small, Connector_Coaxial:U.FL_Molex_MCRF_73412-0110_Vertical, symbol Connector:Conn_Coaxial_Small
- removed TP1, TP2: TestPoint, symbol Connector:TestPoint
- removed U16: 1042240820, 1042240820:1042240820_MOL, symbol 1042240820:1042240820
- removed U18: BG95M3LA-64-SGNS, Quectel_BG95M3LA:BG95_QWS, symbol Quectel_BG95M3LA:BG95M3LA-64-SGNS
- added C81: 10uF, Capacitor_SMD:C_0805_2012Metric, symbol Device:C
- C59, C60, C61, C62, C63, C64, C68: value 100n -> 100nF
Connections:
- net +3.3V: now also C4.1, C5.1, C59.1, C60.1, C61.1, C62.1, C63.1, C64.1, C65.1, C67.1, C68.1, R36.1, U1.5 (OUT), U14.8 (VCC), U15.1 (IOVDD), U15.10 (IOVDD), U15.22 (IOVDD), U15.33 (IOVDD), U15.42 (IOVDD), U15.43 (ADC_AVDD), U15.44 (VREG_IN), U15.48 (USB_VDD), U15.49 (IOVDD)
- net +3.3V_AUX1: now also C81.1
- net +3V3: no longer C4.1, C5.1, C59.1, C60.1, C61.1, C62.1, C63.1, C64.1, C65.1, C67.1, C68.1, R36.1, U1.5 (OUT), U14.8 (VCC), U15.1 (IOVDD), U15.10 (IOVDD), U15.22 (IOVDD), U15.33 (IOVDD), U15.42 (IOVDD), U15.43 (ADC_AVDD), U15.44 (VREG_IN), U15.48 (USB_VDD), U15.49 (IOVDD)
- net BUTTON_R1: now also U15.16 (GPIO13); no longer U15.13 (GPIO10)
- net BUTTON_R2: now also U15.17 (GPIO14); no longer U15.14 (GPIO11)
- net GND: now also C81.2
- net SPI1 MISO_C: now reaches J3.20
- net SPI1 MISO_C: now also J2.20, J3.5, J9.20, J9.5
- net SPI1 MOSI_C: now reaches J3.21
- net SPI1 MOSI_C: now also J2.21, J3.6, J9.21
- net SPI1 SCK_C: now reaches J3.22
- net SPI1 SCK_C: now also J2.22, J3.7, J9.22, J9.7
- net SPI1 MISO: now reaches J2.5
- net SPI1 MISO: now also J8.20, J8.5, U15.15 (GPIO12)
- net SPI1 MOSI : now reaches J2.6
- net SPI1 MOSI : now also J8.21, J8.6, U15.14 (GPIO11)
- net SPI1 SCK: now reaches J2.7
- net SPI1 SCK: now also J8.22, J8.7, U15.13 (GPIO10)
- net SPI1 MOSI _C: now reaches J9.6
Other:
- note added: "SPI1 Bus"
- note removed: "Cell Module"
- moved on the sheet: C57, C58, C59, C60, C61, C62, C63, C64, C65, C66, C67, C68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

Commit message: routing...
Parts:
- removed C78, C79, C80: 1uF, Capacitor_SMD:C_0603_1608Metric, symbol Device:C
- removed U19: TPS7A0533PDBV, Package_TO_SOT_SMD:SOT-23-5, symbol Regulator_Linear:TPS7A0533PDBV
Connections:
- net EYESPI_SCL: now also J2.16; no longer J2.1
- net EYESPI_SDA: now also J2.1; no longer J2.16
- net I2C1_SCL_C: now also J3.16; no longer J3.1
- net I2C1_SDA_C: now also J3.1; no longer J3.16
- net SPI1 MISO: now also J2.26, J8.26; no longer J8.20
- net SPI1 MISO_C: now also J3.26, J9.26; no longer J2.20, J3.20, J9.20
- net SPI1 MOSI_C: now also J3.25, J9.25; no longer J2.21, J3.21, J9.21
- net SPI1 SCK: now also J2.24, J8.24; no longer J8.22
- net SPI1 SCK_C: now also J3.24, J9.24; no longer J2.22, J3.22, J9.22
- net SPI1 MOSI: now reaches J2.25
- net SPI1 MOSI: now also J2.6, J8.25, J8.6, U15.14 (GPIO11)
- removed net SPI1 MOSI : J2.6, J8.21, J8.6, U15.14 (GPIO11)
Other:
- note removed: "Cell Radio"

Commit message: more routing
Parts:
- added R46: 100k, Resistor_SMD:R_0603_1608Metric, symbol Device:R
Connections:
- net +3.3V_AUX2_C: now also U13.1 (VCC)
- net +3.3V_C: now also R46.2
- net GND_C: now also U13.3 (GND)
- net INPUT_INT: now also J2.9, J8.9; no longer U7.22 (~{INT})
- net RESET: no longer U7.24 (~{RESET})
- net LID_SENSE: now reaches U13.2 (OUTPUT)
- net LID_SENSE: now also U7.12 (P1_2)
- net INPUT_INT_C: now reaches J3.9
- net INPUT_INT_C: now also J9.9, U7.22 (~{INT})
- new net: R46.1, U7.24 (~{RESET})
Other:
- moved on the sheet: TH1
