File: PortaPi_R1/PortaPi_R1.kicad_pcb (KiCad board)
At the start: 2 copper layers, 12 parts, among them J1 Raspberry_Pi_2_3, J4 FPC 0.5mmP 18 Pin, U1 BQ24072RGT, U2 TPS61252DSG, U3 LTC2942, U4 BME680, U5 TPS7A0533PDBV, U6 CH340C, U7 RFM95W-915S2, U8 PCM5102A

Commit message: lots of new work and features
Parts:
- added AE1: Antenna, RF_Antenna:Texas_SWRA416_868MHz_915MHz, F.Cu at (84.3, 99.3)
- added AE2: Antenna, RF_Antenna:Pulse_W3000, F.Cu at (103.3, 124.9)
- added C10: 10uF, Capacitor_SMD:C_0805_2012Metric, F.Cu at (76.1, 81.6)
- added C11: 100pF, Capacitor_SMD:C_0603_1608Metric, F.Cu at (54.2, 110.3)
- added C12: 100pF, Capacitor_SMD:C_0603_1608Metric, F.Cu at (54.2, 112.8)
- added C13: 100pF, Capacitor_SMD:C_0603_1608Metric, F.Cu at (54.2, 115.3)
- added C14: 22uF, Capacitor_SMD:C_0805_2012Metric, F.Cu at (76.1, 84.6)
- added C15: 22uF, Capacitor_SMD:C_0805_2012Metric, F.Cu at (76.1, 87.6)
- added C16: 1uF, Capacitor_SMD:C_0603_1608Metric, F.Cu at (54.2, 117.8)
- added C17: 1uF, Capacitor_SMD:C_0603_1608Metric, F.Cu at (54.2, 120.3)
- added C18: 1uF, Capacitor_SMD:C_0603_1608Metric, F.Cu at (58.2, 97.8)
- added C19: 10uF, Capacitor_SMD:C_0805_2012Metric, F.Cu at (76.1, 90.6)
- added C2: 1uF, Capacitor_SMD:C_0603_1608Metric, F.Cu at (54.2, 97.8)
- added C20: 22uF, Capacitor_SMD:C_0805_2012Metric, F.Cu at (80.6, 72.5)
- added C22: 100nF, Capacitor_SMD:C_0603_1608Metric, F.Cu at (58.2, 100.3)
- added C23: 100nF, Capacitor_SMD:C_0603_1608Metric, F.Cu at (58.2, 102.8)
- added C24: 100pF, Capacitor_SMD:C_0603_1608Metric, F.Cu at (58.2, 105.3)
- added C25: 1uF, Capacitor_SMD:C_0805_2012Metric, F.Cu at (80.6, 75.6)
- added C26: 1uF, Capacitor_SMD:C_0805_2012Metric, F.Cu at (80.6, 78.6)
- added C27: 1uF, Capacitor_SMD:C_0805_2012Metric, F.Cu at (80.6, 81.6)
- added C28: 1uF, Capacitor_SMD:C_0603_1608Metric, F.Cu at (58.2, 107.8)
- added C29: 1uF, Capacitor_SMD:C_0603_1608Metric, F.Cu at (58.2, 110.3)
- added C3: 4.7uF, Capacitor_SMD:C_0805_2012Metric, F.Cu at (76.1, 72.5)
- added C30: 1uF, Capacitor_SMD:C_0603_1608Metric, F.Cu at (58.2, 112.8)
- added C31: 1uF, Capacitor_SMD:C_0805_2012Metric, F.Cu at (80.6, 84.6)
- added C32: 10uF, Capacitor_SMD:C_0805_2012Metric, F.Cu at (80.6, 87.6)
- added C33: ~, Capacitor_SMD:C_0805_2012Metric, F.Cu at (80.6, 90.6)
- added C34: ~, Capacitor_SMD:C_0805_2012Metric, F.Cu at (85.0, 72.5)
- added C35: 1uF, Capacitor_SMD:C_0805_2012Metric, F.Cu at (85.0, 75.6)
- added C36: 1uF, Capacitor_SMD:C_0805_2012Metric, F.Cu at (85.0, 78.6)
- added C37: 100nF, Capacitor_SMD:C_0805_2012Metric, F.Cu at (85.0, 81.6)
- added C38: 100nF, Capacitor_SMD:C_0805_2012Metric, F.Cu at (85.0, 84.6)
- added C39: 100nF, Capacitor_SMD:C_0805_2012Metric, F.Cu at (85.0, 87.6)
- added C4: 10uF, Capacitor_SMD:C_0805_2012Metric, F.Cu at (76.1, 75.6)
- added C40: 100nF, Capacitor_SMD:C_0805_2012Metric, F.Cu at (85.0, 90.6)
- added C41: 100nF, Capacitor_SMD:C_0805_2012Metric, F.Cu at (89.5, 72.5)
- added C42: 220pf, Capacitor_SMD:C_0805_2012Metric, F.Cu at (89.5, 75.6)
- added C43: 220pf, Capacitor_SMD:C_0805_2012Metric, F.Cu at (89.5, 78.6)
- added C44: 1uF, Capacitor_SMD:C_0805_2012Metric, F.Cu at (89.5, 81.6)
- added C45: 1uF, Capacitor_SMD:C_0603_1608Metric, F.Cu at (58.2, 115.3)
- added C46: 1uF, Capacitor_SMD:C_0603_1608Metric, F.Cu at (58.2, 117.8)
- added C47: 1uF, Capacitor_SMD:C_0603_1608Metric, F.Cu at (58.2, 120.3)
- added C48: 100nF, Capacitor_SMD:C_0603_1608Metric, F.Cu at (62.2, 97.8)
- added C49: 10uF, Capacitor_SMD:C_0805_2012Metric, F.Cu at (89.5, 84.6)
- added C5: 10uF, Capacitor_SMD:C_0805_2012Metric, F.Cu at (76.1, 78.6)
- added C50: 27p, Capacitor_SMD:C_0402_1005Metric, F.Cu at (93.2, 72.0)
- added C51: 27p, Capacitor_SMD:C_0402_1005Metric, F.Cu at (93.2, 74.0)
- added C52: 100n, Capacitor_SMD:C_0402_1005Metric, F.Cu at (93.2, 76.0)
- added C53: 100n, Capacitor_SMD:C_0402_1005Metric, F.Cu at (93.2, 77.9)
- added C54: 100n, Capacitor_SMD:C_0402_1005Metric, F.Cu at (93.2, 79.9)
- added C55: 1u, Capacitor_SMD:C_0402_1005Metric, F.Cu at (93.2, 81.9)
- added C56: 100n, Capacitor_SMD:C_0402_1005Metric, F.Cu at (96.0, 72.0)
- added C57: 1u, Capacitor_SMD:C_0402_1005Metric, F.Cu at (96.0, 74.0)
- added C58: 100n, Capacitor_SMD:C_0402_1005Metric, F.Cu at (96.0, 76.0)
- added C59: 100n, Capacitor_SMD:C_0402_1005Metric, F.Cu at (96.0, 77.9)
- added C6: 100nF, Capacitor_SMD:C_0603_1608Metric, F.Cu at (54.2, 100.3)
- added C60: 100n, Capacitor_SMD:C_0402_1005Metric, F.Cu at (96.0, 79.9)
- added C61: 100n, Capacitor_SMD:C_0402_1005Metric, F.Cu at (96.0, 81.9)
- added C62: 100n, Capacitor_SMD:C_0402_1005Metric, F.Cu at (98.9, 72.0)
- added C63: 100n, Capacitor_SMD:C_0402_1005Metric, F.Cu at (98.9, 74.0)
- added C64: 100nF, Capacitor_SMD:C_0603_1608Metric, F.Cu at (62.2, 100.3)
- added C65: 100nF, Capacitor_SMD:C_0603_1608Metric, F.Cu at (62.2, 102.8)
- added C66: 120nF, Capacitor_SMD:C_0603_1608Metric, F.Cu at (62.2, 105.3)
- added C67: 6.8nF, Capacitor_SMD:C_0603_1608Metric, F.Cu at (62.2, 107.8)
- added C7: 100nF, Capacitor_SMD:C_0603_1608Metric, F.Cu at (54.2, 102.8)
- added C8: 100pF, Capacitor_SMD:C_0603_1608Metric, F.Cu at (54.2, 105.3)
- added C9: 100nF, Capacitor_SMD:C_0603_1608Metric, F.Cu at (54.2, 107.8)
- added Cr1: 100nF, Capacitor_SMD:C_0603_1608Metric, F.Cu at (62.2, 110.3)
- added Cr2: 100nF, Capacitor_SMD:C_0603_1608Metric, F.Cu at (62.2, 112.8)
- added Cr3: 100nF, Capacitor_SMD:C_0603_1608Metric, F.Cu at (62.2, 115.3)
- added Cr4: 100nF, Capacitor_SMD:C_0603_1608Metric, F.Cu at (62.2, 117.8)
- added Cr5: 100nF, Capacitor_SMD:C_0603_1608Metric, F.Cu at (62.2, 120.3)
- added Cr6: 100nF, Capacitor_SMD:C_0603_1608Metric, F.Cu at (66.2, 97.8)
- added Cr7: 100nF, Capacitor_SMD:C_0603_1608Metric, F.Cu at (66.2, 100.3)
- added J2: USB_C_Receptacle, Connector_USB:USB_C_Receptacle_GCT_USB4105-xx-A_16P_TopMnt_Horizontal, F.Cu at (58.0, 126.9)
- added J7: Conn_01x02, Connector_PinHeader_2.54mm:PinHeader_1x02_P2.54mm_Vertical, F.Cu at (94.5, 127.0)
- added L2: ~, Inductor_SMD:L_0805_2012Metric, F.Cu at (47.3, 130.0)
- added R1: 1.18k, Resistor_SMD:R_0603_1608Metric, F.Cu at (66.2, 102.8)
- added R10: 243k, Resistor_SMD:R_0603_1608Metric, F.Cu at (70.2, 97.8)
- added R11: 1M, Resistor_SMD:R_0603_1608Metric, F.Cu at (70.2, 100.3)
- added R15: 5.1k, Resistor_SMD:R_0603_1608Metric, F.Cu at (70.2, 102.8)
- added R16: 5.1k, Resistor_SMD:R_0603_1608Metric, F.Cu at (70.2, 105.3)
- added R17: 20k, Resistor_SMD:R_0603_1608Metric, F.Cu at (70.2, 107.8)
- added R18: 1k, Resistor_SMD:R_0603_1608Metric, F.Cu at (70.2, 110.3)
- added R19: 20k, Resistor_SMD:R_0603_1608Metric, F.Cu at (70.2, 112.8)
- added R2: 1.13k, Resistor_SMD:R_0603_1608Metric, F.Cu at (66.2, 105.3)
- added R20: 1k, Capacitor_SMD:C_0402_1005Metric, F.Cu at (98.9, 76.0)
- added R21: DNF, Capacitor_SMD:C_0402_1005Metric, F.Cu at (98.9, 77.9)
- added R22: 1k, Capacitor_SMD:C_0402_1005Metric, F.Cu at (98.9, 79.9)
- added R23: 100k, Resistor_SMD:R_0603_1608Metric, F.Cu at (70.2, 115.3)
- added R24: 100k, Resistor_SMD:R_0603_1608Metric, F.Cu at (70.2, 117.8)
- added R4: 10k, Resistor_SMD:R_0603_1608Metric, F.Cu at (66.2, 107.8)
- added R5: 10k, Resistor_SMD:R_0603_1608Metric, F.Cu at (66.2, 110.3)
- added R6: 5.1k, Resistor_SMD:R_0603_1608Metric, F.Cu at (66.2, 112.8)
- added R7: 5.1k, Resistor_SMD:R_0603_1608Metric, F.Cu at (66.2, 115.3)
- added R8: 10k, Resistor_SMD:R_0603_1608Metric, F.Cu at (66.2, 117.8)
- added R9: 768k, Resistor_SMD:R_0603_1608Metric, F.Cu at (66.2, 120.3)
- added TH1: 10k, Resistor_SMD:R_0603_1608Metric, F.Cu at (70.2, 120.3)
- added U10: W25Q128JVS, Package_SO:SOIC-8_5.23x5.23mm_P1.27mm, F.Cu at (105.5, 86.0)
- added U12: TPS7A0533PDBV, Package_TO_SOT_SMD:SOT-23-5, F.Cu at (94.8, 117.8)
- added U13: BG95M3LA-64-SGNS, Quectel_BG95M3LA:BG95_QWS, F.Cu at (63.0, 82.8)
- added U14: TPS7A0533PDBV, Package_TO_SOT_SMD:SOT-23-5, F.Cu at (94.8, 122.4)
- added U15: RP2040, RP2040_minimal:RP2040-QFN-56, F.Cu at (68.5, 126.2)
- added U16: BNO055, Package_LGA:LGA-28_5.2x3.8mm_P0.5mm, F.Cu at (77.5, 127.8)
- added U9: PCAL6416AHF, Package_SO:SOIC-24W_7.5x15.4mm_P1.27mm, F.Cu at (103.8, 114.7)
- added Y1: ABLS-12.000MHZ-B4-T, RP2040_minimal:Crystal_SMD_HC49-US, F.Cu at (102.6, 102.9)
- U7: value RFM95W-915S2 -> RAK3172; footprint RF_Module:HOPERF_RFM9XW_SMD -> RAK3172:RAK3172_RAK
- U8: value PCM5102A -> TLV320AIC3101IRHBR; footprint Package_SO:TSSOP-20_4.4x6.5mm_P0.65mm -> TI_TLV320AIC3101:RHB32_3P45X3P45
- moved U4 60.5 mm to (47.5, 126.3)
- moved U7 37.4 mm to (83.0, 115.5)
- moved J1 37.3 mm to (49.9, 73.4)
- moved U6 29.3 mm to (104.5, 76.9)
- moved U8 27.2 mm to (95.4, 86.8)
- moved U2 22.0 mm to (83.2, 130.4)
- moved U1 19.2 mm to (89.2, 127.5)
- moved U3 10.9 mm to (83.9, 126.7)
- moved D3 9.73 mm to (94.8, 108.5)
- moved U5 9.73 mm to (94.8, 113.2)
- moved J4 5.56 mm to (103.0, 95.0)
Connections:
- J1 pad 13: unconnected-(J1-GPIO27-Pad13) -> /SWCLK
- J1 pad 15: unconnected-(J1-GPIO22-Pad15) -> /LoRaUART_TX
- J1 pad 16: unconnected-(J1-GPIO23-Pad16) -> /LoRaUART_RX
- J1 pad 32: /EYESPI_LITE -> unconnected-(J1-PWM0/GPIO12-Pad32)
- J1 pad 33: unconnected-(J1-PWM1/GPIO13-Pad33) -> /EYESPI_LITE
- J1 pad 37: unconnected-(J1-GPIO26-Pad37) -> /SWD
- J1 pad 7: unconnected-(J1-GCLK0/GPIO4-Pad7) -> /I2S_MCLK
- U7 pad 1: GND -> /LoRaUART_RX
- U7 pad 10: GND -> unconnected-(U7-PA11/I2C_SDA-Pad10)
- U7 pad 11: unconnected-(U7-DIO3-Pad11) -> GND
- U7 pad 12: unconnected-(U7-DIO4-Pad12) -> Net-(U7-RF)
- U7 pad 13: +3.3VA -> unconnected-(U7-PA7/SPI1_MOSI-Pad13)
- U7 pad 2: unconnected-(U7-MISO-Pad2) -> /LoRaUART_TX
- U7 pad 8: GND -> unconnected-(U7-PA14/SWCLK-Pad8)
- U8 pad 1: unconnected-(U8-CPVDD-Pad1) -> /I2S_MCLK
- U8 pad 14: unconnected-(U8-DIN-Pad14) -> /HP_MIC
- U8 pad 15: /I2S_LRCLK -> Net-(U8-MICBIAS)
- U8 pad 16: unconnected-(U8-FMT-Pad16) -> Net-(U8-MIC2R/LINE2R)
- U8 pad 17: unconnected-(U8-XSMT-Pad17) -> GND
- U8 pad 18: unconnected-(U8-LDOO-Pad18) -> +3.3VA
- U8 pad 19: unconnected-(U8-DGND-Pad19) -> Net-(U8-HPLOUT)
- U8 pad 2: unconnected-(U8-CAPP-Pad2) -> /I2S_BC
- U8 pad 3: unconnected-(U8-CPGND-Pad3) -> /I2S_LRCLK
- U8 pad 4: unconnected-(U8-CAPM-Pad4) -> /I2S_TXD
- U8 pad 5: unconnected-(U8-VNEG-Pad5) -> /I2S_RXD
- U8 pad 6: unconnected-(U8-OUTL-Pad6) -> GND
- U8 pad 7: unconnected-(U8-OUTR-Pad7) -> +3.3VA
- U8 pad 8: unconnected-(U8-AVDD-Pad8) -> /EYESPI_SCL
- U8 pad 9: unconnected-(U8-AGND-Pad9) -> /EYESPI_SDA

Commit message: starting layout
Parts:
- removed U6: CH340C, Package_SO:SOIC-16_3.9x9.9mm_P1.27mm
- removed U9: PCAL6416AHF, Package_SO:SOIC-24W_7.5x15.4mm_P1.27mm
- added H1: MountingHole_Pad, MountingHole:MountingHole_2.5mm_Pad_Via, F.Cu at (125.6, 78.8)
- added H2: MountingHole_Pad, MountingHole:MountingHole_2.5mm_Pad_Via, F.Cu at (204.5, 79.9)
- added H3: MountingHole_Pad, MountingHole:MountingHole_2.5mm_Pad_Via, F.Cu at (205.2, 122.6)
- added H4: MountingHole_Pad, MountingHole:MountingHole_2.5mm_Pad_Via, F.Cu at (127.0, 120.4)
- added J8: DF40HC3.0-30DS-0.4V51, DF40HC:CONN_30DS-0.4V51, F.Cu at (124.0, 99.0)
- added J9: DF40HC3.0-30DS-0.4V51, DF40HC:CONN_30DS-0.4V51, F.Cu at (205.0, 99.0)
- added R25: 22, Capacitor_SMD:C_0402_1005Metric, F.Cu at (281.1, 104.1)
- added R26: 22, Capacitor_SMD:C_0402_1005Metric, F.Cu at (283.9, 94.2)
- added R27: 22, Capacitor_SMD:C_0402_1005Metric, F.Cu at (283.9, 96.2)
- added R28: 22, Capacitor_SMD:C_0402_1005Metric, F.Cu at (283.9, 98.2)
- added R29: 22, Capacitor_SMD:C_0402_1005Metric, F.Cu at (283.9, 100.1)
- added R30: 22, Capacitor_SMD:C_0402_1005Metric, F.Cu at (283.9, 102.1)
- added REF**: OSHW-Logo2_9.8x8mm_SilkScreen, Symbol:OSHW-Logo2_9.8x8mm_SilkScreen, F.Cu at (124.8, 88.8)
- J1: footprint Connector_PinSocket_2.54mm:PinSocket_2x20_P2.54mm_Vertical -> Module:Raspberry_Pi_Zero_Socketed_THT_FaceDown_MountingHoles
- U15: footprint RP2040_minimal:RP2040-QFN-56 -> Package_DFN_QFN:QFN-56-1EP_7x7mm_P0.4mm_EP3.2x3.2mm
- moved U4 201.5 mm to (248.2, 109.1)
- moved J7 195.5 mm to (284.7, 81.8)
- moved L2 194.2 mm to (240.4, 109.3)
- moved D3 192.7 mm to (281.4, 60.5)
- moved U12 192.7 mm to (281.4, 69.8)
- moved U14 192.7 mm to (281.4, 74.4)
- moved U5 192.7 mm to (281.4, 65.2)
- moved AE1 189.0 mm to (264.5, 156.6)
- moved C10 187.5 mm to (263.2, 68.7)
- moved C14 187.5 mm to (263.2, 71.7)
- moved C15 187.5 mm to (263.2, 74.7)
- moved C19 187.5 mm to (263.2, 77.7)
- moved C34 187.5 mm to (272.1, 59.6)
- moved C35 187.5 mm to (272.1, 62.7)
- moved C36 187.5 mm to (272.1, 65.7)
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Connections:
- net Net-(U6-UD+) renamed /USB_DP
- net Net-(U6-UD-) renamed /USB_DM
- J1 pad 15: /LoRaUART_TX -> unconnected-(J1-GPIO22-Pad15)
- J1 pad 16: /LoRaUART_RX -> unconnected-(J1-GPIO23-Pad16)
- U12 pad 3: /EN_3.3LoRa -> /EN_3.3Aux1
- U14 pad 3: /EN_3.3LoRa -> /EN_3.3Aux2
- U15 pad 11: unconnected-(U15-GPIO8-Pad11) -> /EYESPI_SDA
- U15 pad 12: unconnected-(U15-GPIO9-Pad12) -> /EYESPI_SCL
- U15 pad 18: unconnected-(U15-GPIO15-Pad18) -> /EYESPI_TFTCS
- U15 pad 2: unconnected-(U15-GPIO0-Pad2) -> Net-(U15-GPIO0)
- U15 pad 27: unconnected-(U15-GPIO16-Pad27) -> /EYESPI_CARDCS
- U15 pad 28: unconnected-(U15-GPIO17-Pad28) -> /EYESPI_MEMCS
- U15 pad 29: unconnected-(U15-GPIO18-Pad29) -> /EYESPI_TSCS
- U15 pad 3: unconnected-(U15-GPIO1-Pad3) -> Net-(U15-GPIO1)
- U15 pad 30: unconnected-(U15-GPIO19-Pad30) -> /EYESPI_TFTDC
- U15 pad 31: unconnected-(U15-GPIO20-Pad31) -> /EYESPI_TFTRST
- U15 pad 32: unconnected-(U15-GPIO21-Pad32) -> /EYESPI_INT
- U15 pad 34: unconnected-(U15-GPIO22-Pad34) -> /EYESPI_BUSY
- U15 pad 36: unconnected-(U15-GPIO24-Pad36) -> /EYESPI_GPIO1
- U15 pad 37: unconnected-(U15-GPIO25-Pad37) -> /EYESPI_GPIO2
- U15 pad 46: unconnected-(U15-USB_DM-Pad46) -> Net-(U15-USB_DM)
- U15 pad 47: unconnected-(U15-USB_DP-Pad47) -> Net-(U15-USB_DP)
- U15 pad 6: unconnected-(U15-GPIO4-Pad6) -> Net-(U15-GPIO4)
- U15 pad 7: unconnected-(U15-GPIO5-Pad7) -> Net-(U15-GPIO5)
Other:
- board outline added: 91 x 57 mm
- board text added: "2000mAh 9mm thick"
- board text added: "3000mAh 10mm thick"
- board text added: "3000mAh 12mm thick"

Commit message: more routing
Parts:
- added J3: AudioJack4, Connector_Audio:Jack_3.5mm_PJ320D_Horizontal, F.Cu at (127.4, 87.2)
- moved U16 23.0 mm to (229.2, 92.6)
- moved REF** 13.9 mm to (138.5, 91.0)
- moved U15 13.5 mm to (164.5, 85.7), turned to 180 degrees
- moved J4 8.44 mm to (164.5, 75.0)
- moved U7 7.26 mm to (144.5, 79.3)
- moved H3 2.91 mm to (204.0, 120.0)
- moved J2 1.96 mm to (123.0, 111.0)
- moved H2 1.94 mm to (204.0, 78.0)
- moved H4 1.07 mm to (126.0, 120.0)
- moved H1 0.84 mm to (126.0, 78.0)

Commit message: placing and routing
Parts:
- removed C11: 100pF, Capacitor_SMD:C_0603_1608Metric
- removed C4: 10uF, Capacitor_SMD:C_0805_2012Metric
- removed Cr1: 100nF, Capacitor_SMD:C_0603_1608Metric
- removed the REF** at (138.5, 91.0)
- added BT1: Battery_Cell, Connector_JST:JST_PH_S2B-PH-SM4-TB_1x02-1MP_P2.00mm_Horizontal, B.Cu at (131.6, 84.8)
- added C1: 4.7uF, Capacitor_SMD:C_0805_2012Metric, F.Cu at (139.2, 84.8)
- added D1: LED, LED_SMD:LED_0603_1608Metric, F.Cu at (130.2, 72.8)
- added D2: LED, LED_SMD:LED_0603_1608Metric, F.Cu at (131.8, 72.8)
- added F1: 1.5 A, Resistor_SMD:R_0603_1608Metric, F.Cu at (138.2, 87.4)
- added FB1: FerriteBead_Small, Resistor_SMD:R_0603_1608Metric, F.Cu at (154.0, 80.5)
- added L1: 1uH, Inductor_SMD:L_Bourns-SRN4018, F.Cu at (139.2, 80.9)
- added R3: 100m, Resistor_SMD:R_0603_1608Metric, F.Cu at (134.5, 84.7)
- added SW1: SW_SPST, Button_Switch_THT:SW_Tactile_SPST_Angled_PTS645Vx31-2LFS, F.Cu at (136.6, 73.4)
- added SW2: SW_Slide_DPDT, Button_Switch_SMD:SW_SPDT_PCM12, F.Cu at (152.2, 72.2)
- added SW3: SW_SPST, Button_Switch_THT:SW_Tactile_SPST_Angled_PTS645Vx31-2LFS, B.Cu at (143.3, 73.4)
- added SW4: SW_SPST, Button_Switch_THT:SW_Tactile_SPST_Angled_PTS645Vx31-2LFS, B.Cu at (191.1, 73.4)
- added SW5: SW_SPST, Button_Switch_THT:SW_Tactile_SPST_Angled_PTS645Vx31-2LFS, F.Cu at (188.8, 73.4)
- C50, C51: value 27p -> 27pf
- R22: value 1k -> 500
- TH1, U13: moved to B.Cu
- Y1: value ABLS-12.000MHZ-B4-T -> ABM3-12.000MHZ-D2Y-T; footprint RP2040_minimal:Crystal_SMD_HC49-US -> Crystal:Crystal_SMD_5032-4Pin_5.0x3.2mm
- moved U12 177.5 mm to (103.8, 68.0)
- moved U14 177.5 mm to (103.8, 72.6)
- moved C49 177.5 mm to (99.0, 69.9)
- moved C36 175.2 mm to (103.9, 114.8)
- moved C39 175.2 mm to (103.9, 123.8)
- moved C40 175.2 mm to (103.9, 126.8)
- moved C41 175.2 mm to (108.3, 108.8)
- moved C42 175.2 mm to (108.3, 111.8)
- moved C43 175.2 mm to (108.3, 114.8)
- moved C44 175.2 mm to (108.3, 117.8)
- moved C25 175.2 mm to (99.5, 111.8)
- moved C26 175.2 mm to (99.5, 114.8)
- moved C27 175.2 mm to (99.5, 117.8)
- moved C31 175.2 mm to (99.5, 120.8)
- moved C32 175.2 mm to (99.5, 123.8)
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Routing:
- net /EYESPI_GPIO2: track 0.00 -> 7.21 mm
- net /EYESPI_GPIO1: track 0.00 -> 6.84 mm
- net /EYESPI_BUSY: track 0.00 -> 6.30 mm
- net /EYESPI_INT: track 0.00 -> 5.76 mm
- net /EYESPI_CARDCS: track 0.00 -> 5.41 mm
- net /EYESPI_MEMCS: track 0.00 -> 4.93 mm
- net /EYESPI_TSCS: track 0.00 -> 4.64 mm
Other:
- copper layers 2 -> 4

Commit message: routing work
Parts:
- added C11: 220pf, Capacitor_SMD:C_0805_2012Metric, F.Cu at (81.6, 100.6)
- added C21: 1uF, Capacitor_SMD:C_0805_2012Metric, F.Cu at (81.6, 103.6)
- added C4: 220pf, Capacitor_SMD:C_0805_2012Metric, F.Cu at (81.6, 97.6)
- added C68: 100nF, Capacitor_SMD:C_0805_2012Metric, F.Cu at (81.6, 106.6)
- added C69: 100nF, Capacitor_SMD:C_0805_2012Metric, F.Cu at (81.6, 109.6)
- added C70: 100nF, Capacitor_SMD:C_0805_2012Metric, F.Cu at (81.6, 112.6)
- added Cr1: 100nF, Capacitor_SMD:C_0603_1608Metric, F.Cu at (94.2, 97.3)
- added D4: ESDA5V3SC5, Package_TO_SOT_SMD:SOT-23-5, F.Cu at (109.0, 140.2)
- added R31: 20k, Resistor_SMD:R_0603_1608Metric, F.Cu at (94.2, 99.9)
- added REF**: AltoidsTinBoundary, AltoidsTin:AltoidsTinBoundary, F.Cu at (144.5, 56.5)
- added SW10: SW_SPST, Button_Switch_SMD:SW_SPST_SKQG_WithoutStem, F.Cu at (120.9, 69.5)
- added SW11: SW_SPST, Button_Switch_SMD:SW_SPST_SKQG_WithoutStem, F.Cu at (130.4, 42.5)
- added SW12: SW_SPST, Button_Switch_SMD:SW_SPST_SKQG_WithoutStem, F.Cu at (130.4, 49.2)
- added SW13: SW_SPST, Button_Switch_SMD:SW_SPST_SKQG_WithoutStem, F.Cu at (130.4, 56.0)
- added SW14: SW_SPST, Button_Switch_SMD:SW_SPST_SKQG_WithoutStem, F.Cu at (130.4, 62.8)
- added SW15: SW_SPST, Button_Switch_SMD:SW_SPST_SKQG_WithoutStem, F.Cu at (130.4, 69.5)
- added SW6: SW_SPST, Button_Switch_SMD:SW_SPST_SKQG_WithoutStem, F.Cu at (120.9, 42.5)
- added SW7: SW_SPST, Button_Switch_SMD:SW_SPST_SKQG_WithoutStem, F.Cu at (120.9, 49.2)
- added SW8: SW_SPST, Button_Switch_SMD:SW_SPST_SKQG_WithoutStem, F.Cu at (120.9, 56.0)
- added SW9: SW_SPST, Button_Switch_SMD:SW_SPST_SKQG_WithoutStem, F.Cu at (120.9, 62.8)
- added U11: PAM8302AAD, Package_SO:SOP-8_3.9x4.9mm_P1.27mm, F.Cu at (88.0, 106.0)
- added U6: PAM8302AAD, Package_SO:SOP-8_3.9x4.9mm_P1.27mm, F.Cu at (88.0, 99.4)
- C52: footprint Capacitor_SMD:C_0402_1005Metric -> Capacitor_SMD:C_0603_1608Metric
- R22: value 500 -> 1k
- moved C52 135.1 mm to (140.6, 109.1), turned to 180 degrees
- moved C56 130.4 mm to (149.4, 114.1), turned to -135 degrees
- moved C59 126.6 mm to (151.6, 103.5), turned to 45 degrees
- moved C58 126.1 mm to (152.7, 110.8), turned to 45 degrees
- moved C20 121.7 mm to (158.7, 113.8), turned to 90 degrees
- moved C47 116.3 mm to (126.9, 109.8), turned to 180 degrees
- moved C46 114.6 mm to (129.2, 109.2), turned to 90 degrees
- moved C45 114.4 mm to (129.2, 106.2), turned to -90 degrees
- moved C29 114.4 mm to (131.8, 109.8), turned to 180 degrees
- moved C28 111.5 mm to (134.2, 105.1), turned to -90 degrees
- moved C30 110.9 mm to (134.2, 108.1), turned to 90 degrees
- moved C18 110.7 mm to (139.2, 105.5), turned to 90 degrees
- moved C19 108.7 mm to (160.7, 113.8), turned to 90 degrees
- moved C16 101.8 mm to (136.9, 103.8), turned to 180 degrees
- moved C17 99.3 mm to (139.9, 107.8)
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Routing:
- net /EYESPI_GPIO2: track 7.21 -> 0.00 mm
- net /EYESPI_GPIO1: track 6.84 -> 0.00 mm
- net /EYESPI_BUSY: track 6.30 -> 0.00 mm
- net /EYESPI_INT: track 5.76 -> 0.00 mm
- net /EYESPI_CARDCS: track 5.41 -> 0.00 mm
- net /EYESPI_MEMCS: track 4.93 -> 0.00 mm
- net /EYESPI_TSCS: track 4.64 -> 0.00 mm

Commit message: lots more routing work
Parts:
- added J11: DF40HC3.0-30DP, DF40C-30DP:SOIC_0DP-0.4V51_HIR, F.Cu at (53.0, 60.0)
- added J12: DF40HC3.0-30DP, DF40C-30DP:SOIC_0DP-0.4V51_HIR, F.Cu at (136.0, 60.0)
- added R32: 20k, Resistor_SMD:R_0603_1608Metric, F.Cu at (33.6, 129.4)
- added R33: 20k, Resistor_SMD:R_0603_1608Metric, F.Cu at (116.0, 44.2)
- added R34: 20k, Resistor_SMD:R_0603_1608Metric, F.Cu at (119.0, 53.2)
- added R35: 20k, Resistor_SMD:R_0603_1608Metric, F.Cu at (54.0, 52.4)
- added R36: 20k, Resistor_SMD:R_0603_1608Metric, F.Cu at (68.4, 50.4)
- added R37: 20k, Resistor_SMD:R_0603_1608Metric, F.Cu at (130.0, 61.0)
- added R38: 20k, Resistor_SMD:R_0603_1608Metric, F.Cu at (119.0, 56.8)
- added R39: 20k, Resistor_SMD:R_0603_1608Metric, F.Cu at (70.4, 53.6)
- added R40: 20k, Resistor_SMD:R_0603_1608Metric, F.Cu at (70.4, 57.6)
- added R41: 20k, Resistor_SMD:R_0603_1608Metric, F.Cu at (93.5, 34.4)
- added R42: 20k, Resistor_SMD:R_0603_1608Metric, F.Cu at (96.0, 34.4)
- added R43: 20k, Resistor_SMD:R_0603_1608Metric, F.Cu at (76.8, 93.6)
- added R44: 20k, Resistor_SMD:R_0603_1608Metric, F.Cu at (112.4, 95.4)
- added R45: 20k, Resistor_SMD:R_0603_1608Metric, F.Cu at (110.8, 95.4)
- added R46: 20k, Resistor_SMD:R_0603_1608Metric, F.Cu at (63.2, 92.8)
- added U9: PCAL6416AHF, Package_DFN_QFN:HVQFN-24-1EP_4x4mm_P0.5mm_EP2.1x2.1mm, F.Cu at (87.1, 53.4)
- C35, C37, C38, C39, C40, C41: footprint Capacitor_SMD:C_0805_2012Metric -> Capacitor_SMD:C_0603_1608Metric
- J1: moved to B.Cu
- R18: footprint Resistor_SMD:R_0603_1608Metric -> Capacitor_SMD:C_0603_1608Metric
- SW10: value SW_SPST -> L; footprint Button_Switch_SMD:SW_SPST_SKQG_WithoutStem -> Button_Switch_THT:SW_PUSH_6mm; moved to B.Cu
- SW11: value SW_SPST -> R; footprint Button_Switch_SMD:SW_SPST_SKQG_WithoutStem -> Button_Switch_THT:SW_PUSH_6mm; moved to B.Cu
- SW12: value SW_SPST -> U; footprint Button_Switch_SMD:SW_SPST_SKQG_WithoutStem -> Button_Switch_THT:SW_PUSH_6mm; moved to B.Cu
- SW13: value SW_SPST -> D; footprint Button_Switch_SMD:SW_SPST_SKQG_WithoutStem -> Button_Switch_THT:SW_PUSH_6mm; moved to B.Cu
- SW14, SW15: footprint Button_Switch_SMD:SW_SPST_SKQG_WithoutStem -> Button_Switch_THT:SW_PUSH_6mm; moved to B.Cu
- SW6: value SW_SPST -> A; footprint Button_Switch_SMD:SW_SPST_SKQG_WithoutStem -> Button_Switch_THT:SW_PUSH_6mm; moved to B.Cu
- SW7: value SW_SPST -> X; footprint Button_Switch_SMD:SW_SPST_SKQG_WithoutStem -> Button_Switch_THT:SW_PUSH_6mm; moved to B.Cu
- SW8: value SW_SPST -> B; footprint Button_Switch_SMD:SW_SPST_SKQG_WithoutStem -> Button_Switch_THT:SW_PUSH_6mm; moved to B.Cu
- SW9: value SW_SPST -> Y; footprint Button_Switch_SMD:SW_SPST_SKQG_WithoutStem -> Button_Switch_THT:SW_PUSH_6mm; moved to B.Cu
- moved AE2 272.3 mm to (-65.6, 87.0)
- moved C33 272.3 mm to (-23.2, 125.6)
- moved C34 272.3 mm to (-18.8, 107.5)
- moved J7 272.3 mm to (-67.3, 130.6)
- moved L2 272.3 mm to (-50.5, 157.2)
- moved R20 272.3 mm to (-9.80, 146.0)
- moved R21 272.3 mm to (-9.80, 148.0)
- moved R28 206.5 mm to (57.8, 107.2), turned to 90 degrees
- moved R27 206.3 mm to (57.8, 109.4), turned to -90 degrees
- moved AE1 203.9 mm to (-2.71, 137.2)
- moved C61 167.2 mm to (91.8, 106.7), turned to 90 degrees
- moved C62 165.0 mm to (96.1, 111.0), turned to -135 degrees
- moved C63 164.4 mm to (96.8, 111.7), turned to -135 degrees
- moved C57 162.9 mm to (95.4, 110.3), turned to -135 degrees
- moved C60 161.6 mm to (97.7, 103.3), turned to 135 degrees
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Connections:
- C11 pad 1: unconnected-(C11-Pad1) -> GND
- C21 pad 1: Net-(U6-VDD) -> +3.3VA
- C4 pad 1: unconnected-(C4-Pad1) -> GND
- C40 pad 1: Net-(U11-IN+) -> /LEFT_LOM_CON
- C41 pad 1: Net-(U11-IN-) -> /LEFT_LOP_CON
- C68 pad 1: Net-(U6-IN+) -> /RIGHT_LOM_CON
- C69 pad 1: Net-(U6-IN-) -> /RIGHT_LOP_CON
- Cr1 pad 1: Net-(U6-VDD) -> +3.3VA
- J8 pad 13: unconnected-(J8-Pad13) -> /LEFT_LOP_CON
- J8 pad 14: unconnected-(J8-Pad14) -> GND
- J8 pad 15: unconnected-(J8-Pad15) -> /EYESPI_SCL
- J8 pad 17: unconnected-(J8-Pad17) -> GND
- J8 pad 18: unconnected-(J8-Pad18) -> /RIGHT_LOM_CON
- J8 pad 19: unconnected-(J8-Pad19) -> +3.3VA
- J8 pad 2: unconnected-(J8-Pad2) -> GND
- J8 pad 28: unconnected-(J8-Pad28) -> /LEFT_LOM_CON
- J8 pad 29: unconnected-(J8-Pad29) -> GND
- J8 pad 3: unconnected-(J8-Pad3) -> /RIGHT_LOP_CON
- J8 pad 30: unconnected-(J8-Pad30) -> /EYESPI_SDA
- J8 pad 4: unconnected-(J8-Pad4) -> /+3.3V_AUX1
- J9 pad 1: unconnected-(J9-Pad1) -> /EYESPI_SCL
- J9 pad 12: unconnected-(J9-Pad12) -> +3.3VA
- J9 pad 14: unconnected-(J9-Pad14) -> GND
- J9 pad 16: unconnected-(J9-Pad16) -> /EYESPI_SDA
- J9 pad 17: unconnected-(J9-Pad17) -> GND
- J9 pad 2: unconnected-(J9-Pad2) -> GND
- J9 pad 27: unconnected-(J9-Pad27) -> /+3.3V_AUX1
- J9 pad 29: unconnected-(J9-Pad29) -> GND
- R17 pad 2: Net-(U8-RIGHT_LOM) -> Net-(U8-LEFT_LOM)
- R19 pad 2: Net-(U8-RIGHT_LOP) -> Net-(U8-LEFT_LOP)
- R31 pad 2: unconnected-(R31-Pad2) -> Net-(U8-RIGHT_LOP)
- SW1 pad 1: unconnected-(SW1-A-Pad1) -> /BUTTON_L2
- SW1 pad 2: unconnected-(SW1-B-Pad2) -> GND
- SW10 pad 1: unconnected-(SW10-A-Pad1) -> /BUTTON_L
- SW10 pad 2: unconnected-(SW10-B-Pad2) -> GND
- SW11 pad 1: unconnected-(SW11-A-Pad1) -> /BUTTON_R
- SW11 pad 2: unconnected-(SW11-B-Pad2) -> GND
- SW12 pad 1: unconnected-(SW12-A-Pad1) -> /BUTTON_U
- SW12 pad 2: unconnected-(SW12-B-Pad2) -> GND
- SW13 pad 1: unconnected-(SW13-A-Pad1) -> /BUTTON_D
- SW13 pad 2: unconnected-(SW13-B-Pad2) -> GND
- SW14 pad 1: unconnected-(SW14-A-Pad1) -> /BUTTON_START
- SW14 pad 2: unconnected-(SW14-B-Pad2) -> GND
- SW15 pad 1: unconnected-(SW15-A-Pad1) -> /BUTTON_SELECT
- SW15 pad 2: unconnected-(SW15-B-Pad2) -> GND
- SW3 pad 1: unconnected-(SW3-A-Pad1) -> /BUTTON_L1
- SW3 pad 2: unconnected-(SW3-B-Pad2) -> GND
- SW4 pad 1: unconnected-(SW4-A-Pad1) -> /BUTTON_R1
- SW4 pad 2: unconnected-(SW4-B-Pad2) -> GND
- SW5 pad 1: unconnected-(SW5-A-Pad1) -> /BUTTON_R2
- SW5 pad 2: unconnected-(SW5-B-Pad2) -> GND
- SW6 pad 1: unconnected-(SW6-A-Pad1) -> /BUTTON_A
- SW6 pad 2: unconnected-(SW6-B-Pad2) -> GND
- SW7 pad 1: unconnected-(SW7-A-Pad1) -> /BUTTON_X
- SW7 pad 2: unconnected-(SW7-B-Pad2) -> GND
- SW8 pad 1: unconnected-(SW8-A-Pad1) -> /BUTTON_B
- SW8 pad 2: unconnected-(SW8-B-Pad2) -> GND
- SW9 pad 1: unconnected-(SW9-A-Pad1) -> /BUTTON_Y
- SW9 pad 2: unconnected-(SW9-B-Pad2) -> GND
- U11 pad 1: /AudioAmp_SD -> +3.3VA
- U11 pad 3: Net-(U11-IN+) -> /LEFT_LOM
- U11 pad 4: Net-(U11-IN-) -> /LEFT_LOP
- U15 pad 13: unconnected-(U15-GPIO10-Pad13) -> /BUTTON_R1
- U15 pad 14: unconnected-(U15-GPIO11-Pad14) -> /BUTTON_R2
- U15 pad 8: unconnected-(U15-GPIO6-Pad8) -> /BUTTON_L1
- U15 pad 9: unconnected-(U15-GPIO7-Pad9) -> /BUTTON_L2
- U6 pad 1: /AudioAmp_SD -> unconnected-(U6-~{SD}-Pad1)
- U6 pad 3: Net-(U6-IN+) -> /RIGHT_LOM
- U6 pad 4: Net-(U6-IN-) -> /RIGHT_LOP
- U6 pad 6: Net-(U6-VDD) -> +3.3VA
- U8 pad 27: unconnected-(U8-LEFT_LOP-Pad27) -> Net-(U8-LEFT_LOP)
- U8 pad 28: unconnected-(U8-LEFT_LOM-Pad28) -> Net-(U8-LEFT_LOM)
Routing:
- net unconnected-(J1-GPIO24-Pad18): vias 0 -> 1
- net unconnected-(J1-GPIO23-Pad16): vias 0 -> 3
- net unconnected-(J1-GPIO22-Pad15): vias 0 -> 2
- net (no net): vias 0 -> 78
Other:
- board size 91 x 57 mm -> 184 x 131 mm
- board text added: "A"
- board text added: "B"
- board text added: "D"
- board text added: "L"
- board text added: "R"
- board text added: "SELECT"
- board text added: "START"
- board text added: "U"
- board text added: "X"
- board text added: "Y"
