File: PortaPi_R1/PortaPi_R1.kicad_pcb (KiCad board)
At the start: 4 copper layers, 184 x 131 mm, 179 parts, among them J1 Raspberry_Pi_2_3, J11 DF40HC3.0-30DP, J12 DF40HC3.0-30DP, J2 USB_C_Receptacle, J3 AudioJack4, J4 FPC 0.5mmP 18 Pin, J7 Conn_01x02, J8 DF40HC3.0-30DS-0.4V51, J9 DF40HC3.0-30DS-0.4V51, SW1 SW_SPST, SW10 L, SW11 R, SW12 U, SW13 D, SW14 SW_SPST, SW15 SW_SPST, SW2 SW_Slide_DPDT, SW3 SW_SPST, SW4 SW_SPST, SW5 SW_SPST, SW6 A, SW7 X, SW8 B, SW9 Y, U1 BQ24072RGT, U10 W25Q128JVS, U11 PAM8302AAD, U12 TPS7A0533PDBV, U13 BG95M3LA-64-SGNS, U14 TPS7A0533PDBV, U15 RP2040, U16 BNO055, U2 TPS61252DSG, U3 LTC2942, U4 BME680, U5 TPS7A0533PDBV, U6 PAM8302AAD, U7 RAK3172, U8 TLV320AIC3101IRHBR, U9 PCAL6416AHF, Y1 ABM3-12.000MHZ-D2Y-T

Commit message: placing work
Parts:
- removed AE1: Antenna, RF_Antenna:Texas_SWRA416_868MHz_915MHz
- removed AE2: Antenna, RF_Antenna:Pulse_W3000
- removed the C33 at (-23.2, 125.6)
- removed the C34 at (-18.8, 107.5)
- removed the J7 at (-67.3, 130.6)
- removed L2: ~, Inductor_SMD:L_0805_2012Metric
- added D5: WS2812, LED_SMD:LED_WS2812_PLCC6_5.0x5.0mm_P1.6mm, B.Cu at (84.7, 79.3)
- added D6: WS2812, LED_SMD:LED_WS2812_PLCC6_5.0x5.0mm_P1.6mm, B.Cu at (91.3, 79.3)
- added D7: WS2812, LED_SMD:LED_WS2812_PLCC6_5.0x5.0mm_P1.6mm, B.Cu at (97.9, 79.3)
- added D8: WS2812, LED_SMD:LED_WS2812_PLCC6_5.0x5.0mm_P1.6mm, B.Cu at (104.2, 79.3)
- added FB2: FerriteBead_Small, Inductor_SMD:L_0603_1608Metric, F.Cu at (72.0, 75.0)
- added FB3: FerriteBead_Small, Inductor_SMD:L_0603_1608Metric, F.Cu at (72.0, 77.5)
- added FB4: FerriteBead_Small, Inductor_SMD:L_0603_1608Metric, F.Cu at (72.0, 70.0)
- added FB5: FerriteBead_Small, Inductor_SMD:L_0603_1608Metric, F.Cu at (72.0, 72.5)
- added J11: Conn_Coaxial_Small, Connector_Coaxial:U.FL_Molex_MCRF_73412-0110_Vertical, F.Cu at (136.6, 103.3)
- added J12: Conn_Coaxial_Small, Connector_Coaxial:U.FL_Molex_MCRF_73412-0110_Vertical, B.Cu at (135.9, 134.5)
- added R30: 0, Resistor_SMD:R_0603_1608Metric, F.Cu at (134.1, 107.8)
- added R31: 0, Resistor_SMD:R_0603_1608Metric, F.Cu at (132.5, 107.8)
- added SW12: BOOT, Button_Switch_SMD:SW_SPST_B3U-1000P-B, F.Cu at (80.7, 113.1)
- added U13: SM351LT, Package_TO_SOT_SMD:SOT-23, F.Cu at (85.5, 72.6)
- added U16: 1042240820, 1042240820:1042240820_MOL, B.Cu at (117.9, 141.2)
- C27: renamed from C36; footprint Capacitor_SMD:C_0805_2012Metric -> Capacitor_SMD:C_0603_1608Metric
- C29: renamed from C25; footprint Capacitor_SMD:C_0805_2012Metric -> Capacitor_SMD:C_0603_1608Metric
- C31: renamed from C68; footprint Capacitor_SMD:C_0805_2012Metric -> Capacitor_SMD:C_0603_1608Metric
- C32: renamed from C70; footprint Capacitor_SMD:C_0805_2012Metric -> Capacitor_SMD:C_0603_1608Metric
- C33: renamed from C69; footprint Capacitor_SMD:C_0805_2012Metric -> Capacitor_SMD:C_0603_1608Metric
- C35: renamed from C31; footprint Capacitor_SMD:C_0805_2012Metric -> Capacitor_SMD:C_0603_1608Metric
- C37: renamed from C26; footprint Capacitor_SMD:C_0805_2012Metric -> Capacitor_SMD:C_0603_1608Metric
- C39: renamed from C27; footprint Capacitor_SMD:C_0805_2012Metric -> Capacitor_SMD:C_0603_1608Metric
- moved R36 100.0 mm to (83.8, 112.7), turned to 90 degrees
- moved R39 99.5 mm to (83.4, 111.2), turned to 180 degrees
- moved C54 85.9 mm to (111.3, 114.4), turned to 180 degrees
- moved C35 45.4 mm to (62.0, 113.1), turned to 90 degrees
- moved C29 42.4 mm to (65.5, 113.2), turned to 90 degrees
- moved C39 38.6 mm to (64.1, 124.2), turned to 180 degrees
- moved C37 36.2 mm to (64.1, 127.2), turned to 180 degrees
- moved R14 29.8 mm to (105.1, 99.7)
- moved C31 29.8 mm to (54.0, 126.2), turned to -90 degrees
- moved C27 27.5 mm to (56.5, 122.9), turned to -90 degrees
- moved R24 26.5 mm to (50.8, 125.6), turned to 90 degrees
- moved C33 26.3 mm to (52.4, 125.6), turned to -90 degrees
- moved C32 25.1 mm to (51.4, 128.0), turned to 180 degrees
- moved C53 25.1 mm to (110.7, 112.6), turned to 180 degrees
- moved R38 22.8 mm to (132.6, 114.2), turned to -90 degrees
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- renumbered C3 to C1, C13 to C10, C9 to C11, C10 to C12, C14 to C13, C15 to C14, C28 to C15, C29 to C16, C30 to C17, C8 to C18, C45 to C19, C46 to C20, C47 to C21, C24 to C22, C6 to C23, C20 to C24, C19 to C25, Cr2 to C26, Cr3 to C28, C16 to C3, C32 to C30, Cr6 to C34, Cr4 to C36, Cr5 to C38, C17 to C4, C21 to C40, C4 to C41, C40 to C42, C11 to C43, C39 to C44, C41 to C45, C38 to C46, C37 to C47, C35 to C48, C44 to C49, C18 to C5, Cr7 to C50, C42 to C51, C43 to C52, C48 to C53, C49 to C54, C22 to C55, C23 to C56, C53 to C57, C54 to C58, C56 to C59, C7 to C6, C58 to C60, C59 to C61, C60 to C62, C61 to C63, C62 to C64, C63 to C65, C55 to C66, C57 to C67, C52 to C68, C65 to C69, C12 to C7, C66 to C70, C67 to C71, C50 to C72, C51 to C73, C64 to C74, Cr1 to C75, C5 to C8, C1 to C9, J2 to J1, J9 to J2, J12 to J3, J1 to J5, J3 to J7, J11 to J9, R3 to R1, R15 to R10, R10 to R11, R33 to R12, R37 to R13, R23 to R14, R34 to R15, R38 to R16, R35 to R17, R39 to R18, R36 to R19, R6 to R2, R40 to R20, R41 to R21, R42 to R22, R32 to R23, R31 to R24, R4 to R25, R5 to R26, R17 to R27, R19 to R28, R18 to R29, R7 to R3, R27 to R32, R28 to R33, R25 to R34, R26 to R35, R21 to R36, R29 to R37, R30 to R38, R20 to R39, R1 to R4, R24 to R40, R22 to R41, R46 to R42, R45 to R44, R44 to R45, R2 to R5, R11 to R6, R9 to R7, R16 to R8, R8 to R9, SW2 to SW1, SW14 to SW10, SW15 to SW11, SW1 to SW13, SW3 to SW14, SW4 to SW15, SW5 to SW16, SW6 to SW2, SW7 to SW3, SW8 to SW4, SW9 to SW5, SW10 to SW6, SW11 to SW7, SW12 to SW8, SW13 to SW9, U5 to U1, U11 to U10, U4 to U11, U7 to U12, U10 to U14, U16 to U17, U13 to U18, U1 to U2, U2 to U3, U12 to U4, U3 to U5, U14 to U6, U9 to U7, U6 to U8, U8 to U9
Connections:
- J2 pad 12: +3.3VA -> +3.3V
- J2 pad 15: unconnected-(J9-Pad15) -> /EYESPI_SCL
- J2 pad 19: unconnected-(J9-Pad19) (its old number) -> +3.3V
- J2 pad 23: unconnected-(J9-Pad23) (its old number) -> +5V
- J2 pad 30: unconnected-(J9-Pad30) -> /EYESPI_SDA
- J2 pad 4: unconnected-(J9-Pad4) (its old number) -> /+3.3V_AUX1
- J2 pad 8: unconnected-(J9-Pad8) -> +5V
- J3 pad 14: unconnected-(J12-Pad14) -> GND
- J3 pad 17: unconnected-(J12-Pad17) -> GND
- J3 pad 2: unconnected-(J12-Pad2) -> GND
- J3 pad 23: unconnected-(J12-Pad23) -> +5V
- J3 pad 29: unconnected-(J12-Pad29) -> GND
- J3 pad 8: unconnected-(J12-Pad8) -> +5V
- J8 pad 1: unconnected-(J8-Pad1) -> /EYESPI_SDA
- J8 pad 12: unconnected-(J8-Pad12) -> +3.3V
- J8 pad 16: unconnected-(J8-Pad16) -> /EYESPI_SCL
- J8 pad 19: +3.3VA -> +3.3V
- J8 pad 23: unconnected-(J8-Pad23) -> +5V
- J8 pad 27: unconnected-(J8-Pad27) -> /+3.3V_AUX1
- J8 pad 8: unconnected-(J8-Pad8) -> +5V
- J9 pad 13: unconnected-(J11-Pad13) -> /LEFT_LOP
- J9 pad 14: unconnected-(J11-Pad14) -> GND
- J9 pad 15: unconnected-(J11-Pad15) -> /EYESPI_SCL
- J9 pad 17: unconnected-(J11-Pad17) -> GND
- J9 pad 18: unconnected-(J11-Pad18) -> /RIGHT_LOM
- J9 pad 2: unconnected-(J11-Pad2) -> GND
- J9 pad 28: unconnected-(J11-Pad28) -> /LEFT_LOM
- J9 pad 29: unconnected-(J11-Pad29) -> GND
- J9 pad 3: unconnected-(J11-Pad3) -> /RIGHT_LOP
- J9 pad 30: unconnected-(J11-Pad30) -> /EYESPI_SDA
- J9 pad 8: unconnected-(J11-Pad8) -> +5V
- U12 pad 10: unconnected-(U7-PA11/I2C_SDA-Pad10) -> /EYESPI_SDA
- U12 pad 9: unconnected-(U7-PA12/I2C_SCL-Pad9) -> /EYESPI_SCL
- U18 pad 3: unconnected-(U13A-GND-Pad3) -> GND
- U18 pad 31: unconnected-(U13A-GND-Pad31) -> GND
- U18 pad 40: unconnected-(U13A-I2C_SCL-Pad40) -> /EYESPI_SCL
- U18 pad 41: unconnected-(U13A-I2C_SDA-Pad41) -> /EYESPI_SDA
- U18 pad 48: unconnected-(U13A-GND-Pad48) -> GND
- U18 pad 50: unconnected-(U13A-GND-Pad50) -> GND
Other:
- board size 184 x 131 mm -> 184.2 x 131 mm
- board text added: "2.0{dblquote} 320x240 Color IPS TFT Display with microSD Card Breakout - ST7789 EYESPI"
- board text added: "2.2{dblquote} 18-bit color TFT LCD display with microSD card breakout - EYESPI Connector"
- board text added: "2.8{dblquote} TFT Touch Shield for Arduino with Capacitive Touch"
- board text added: "Adafruit 2.8{dblquote} and 3.2{dblquote} Color TFT Touchscreen Breakout v2"

Commit message: routing and placinggit add .!
Parts:
- removed D8: WS2812, LED_SMD:LED_WS2812_PLCC6_5.0x5.0mm_P1.6mm
- added C76: 100n, Capacitor_SMD:C_0402_1005Metric, F.Cu at (88.3, 49.8)
- added C77: 100n, Capacitor_SMD:C_0402_1005Metric, F.Cu at (86.1, 49.8)
- added D9: WS2812B, LED_SMD:LED_WS2812B_PLCC4_5.0x5.0mm_P3.2mm, B.Cu at (111.3, 81.8)
- added FID1: Fiducial, Fiducial:Fiducial_1.5mm_Mask3mm, F.Cu at (54.0, 152.5)
- added FID2: Fiducial, Fiducial:Fiducial_1.5mm_Mask3mm, F.Cu at (54.0, 27.0)
- added FID3: Fiducial, Fiducial:Fiducial_1.5mm_Mask3mm, F.Cu at (228.0, 152.5)
- added FID4: Fiducial, Fiducial:Fiducial_1.5mm_Mask3mm, F.Cu at (228.0, 27.0)
- added J10: SpeakerOut, Jumper:SolderJumper-2_P1.3mm_Open_Pad1.0x1.5mm, B.Cu at (87.2, 54.5)
- added J6: SpeakerOut, Jumper:SolderJumper-2_P1.3mm_Open_Pad1.0x1.5mm, B.Cu at (98.9, 53.0)
- C40, C41, C43, C49, C51, C52: footprint Capacitor_SMD:C_0805_2012Metric -> Capacitor_SMD:C_0603_1608Metric
- D5, D6, D7: value WS2812 -> WS2812B; footprint LED_SMD:LED_WS2812_PLCC6_5.0x5.0mm_P1.6mm -> LED_SMD:LED_WS2812B_PLCC4_5.0x5.0mm_P3.2mm
- U13: moved to B.Cu
- moved U13 46.9 mm to (132.0, 78.5), turned to 180 degrees
- moved C49 18.2 mm to (68.6, 70.7), turned to 90 degrees
- moved C52 16.8 mm to (71.7, 75.5), turned to 90 degrees
- moved C41 16.6 mm to (71.7, 72.4), turned to -90 degrees
- moved C43 16.2 mm to (71.7, 69.3), turned to 90 degrees
- moved C51 16.1 mm to (71.7, 78.5), turned to -90 degrees
- moved C40 14.2 mm to (69.4, 77.8)
- moved FB4 9.69 mm to (69.4, 79.3), turned to 180 degrees
- moved R11 9.50 mm to (75.2, 96.2), turned to 90 degrees
- moved FB3 9.50 mm to (69.3, 68.4), turned to 180 degrees
- moved D5 7.41 mm to (77.6, 81.6), turned to 0 degrees
- moved C73 6.45 mm to (106.0, 101.6), turned to 45 degrees
- moved C50 5.71 mm to (69.4, 76.2)
- moved R34 4.14 mm to (103.5, 113.5), turned to 135 degrees
- moved R35 3.41 mm to (104.2, 112.8), turned to 135 degrees
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Connections:
- C4 pad 1: +3.3VA -> +3V3
- C5 pad 1: +3.3VA -> +3V3
- D5 pad 1: Net-(D5-DOUT) -> +5V
- D5 pad 2: unconnected-(D5-DIN-Pad2) -> Net-(D5-DOUT)
- D5 pad 3: unconnected-(D5-VCC-Pad3) -> GND
- D5 pad 4: unconnected-(D5-NC-Pad4) -> Net-(D5-DIN)
- D6 pad 1: Net-(D6-DOUT) -> +5V
- D6 pad 2: Net-(D5-DOUT) -> Net-(D6-DOUT)
- D6 pad 3: unconnected-(D6-VCC-Pad3) -> GND
- D6 pad 4: unconnected-(D6-NC-Pad4) -> Net-(D5-DOUT)
- D7 pad 1: Net-(D7-DOUT) -> +5V
- D7 pad 2: Net-(D6-DOUT) -> unconnected-(D7-DOUT-Pad2)
- D7 pad 3: unconnected-(D7-VCC-Pad3) -> GND
- D7 pad 4: unconnected-(D7-NC-Pad4) -> Net-(D6-DOUT)
- J5 pad 1: +3.3V -> Net-(J5-3V3-Pad1)
- J5 pad 17: +3.3V -> Net-(J5-3V3-Pad1)
- J5 pad 33: /EYESPI_LITE -> unconnected-(J5-PWM1/GPIO13-Pad33)
- U1 pad 5: +3.3VA -> +3V3
- U15 pad 35: unconnected-(U15-GPIO23-Pad35) -> /EYESPI_LITE
- U7 pad 21: unconnected-(U7-V_{DD(P)}-Pad21) -> +3.3V
- U7 pad 23: unconnected-(U7-V_{DD(I2C-bus)}-Pad23) -> +3.3V
- Y1 pad 1: /XIN -> Net-(C73-Pad1)
- Y1 pad 2: Net-(C73-Pad1) -> /XIN
Routing:
- net +5V: track 0.00 -> 31.6 mm
- net +3V3: track 0.00 -> 30.3 mm
- net Net-(C1-Pad1): track 0.00 -> 30.1 mm, vias 0 -> 2
- net /QSPI_SS: track 0.00 -> 23.0 mm, vias 0 -> 2
- net Net-(U3-EN): track 0.00 -> 20.9 mm, vias 0 -> 2
- net +3.3VA: track 0.00 -> 20.0 mm
- net Net-(U9-HPROUT): track 0.00 -> 18.1 mm
- net /QSPI_SD1: track 0.00 -> 18.1 mm, vias 0 -> 2
- net /QSPI_SD2: track 0.00 -> 16.6 mm, vias 0 -> 2
- net /HP_R: track 0.00 -> 16.2 mm
- net Net-(U9-HPLOUT): track 0.00 -> 12.6 mm
- net GND: track 0.00 -> 11.8 mm
- net /EYESPI_GPIO2: track 0.00 -> 10.2 mm
- net /EYESPI_GPIO1: track 0.00 -> 9.87 mm
- net /EYESPI_BUSY: track 0.00 -> 9.70 mm
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- added copper zone on B.Cu, net GND
- added copper zone on F.Cu, net GND
- added copper zone on F.Cu, net Net-(U3-EN)
- added copper zone on F.Cu, net Net-(U3-SW)
- added copper zone on F.Cu, net Net-(U3-VOUT)
Other:
- outline, holes or cut-outs redrawn
