File: PortaPi_R1/PortaPi_R1.kicad_pcb (KiCad board)
At the start: 4 copper layers, 184.2 x 131 mm, 196 parts, among them J1 USB_C_Receptacle, J10 SpeakerOut, J11 Conn_Coaxial_Small, J12 Conn_Coaxial_Small, J2 DF40HC3.0-30DS-0.4V51, J3 DF40HC3.0-30DP, J4 FPC 0.5mmP 18 Pin, J5 Raspberry_Pi_2_3, J6 SpeakerOut, J7 AudioJack4, J8 DF40HC3.0-30DS-0.4V51, J9 DF40HC3.0-30DP, SW1 SW_Slide_DPDT, SW10 SW_SPST, SW11 SW_SPST, SW12 BOOT, SW13 SW_SPST, SW14 SW_SPST, SW15 SW_SPST, SW16 SW_SPST, SW2 A, SW3 X, SW4 B, SW5 Y, SW6 L, SW7 R, SW8 U, SW9 D, U1 TPS7A0533PDBV, U10 PAM8302AAD, U11 BME680, U12 RAK3172, U13 SM351LT, U14 W25Q128JVS, U15 RP2040, U16 1042240820, U17 BNO055, U18 BG95M3LA-64-SGNS, U2 BQ24072RGT, U3 TPS61252DSG, U4 TPS7A0533PDBV, U5 LTC2942, U6 TPS7A0533PDBV, U7 PCAL6416AHF, U8 PAM8302AAD, U9 TLV320AIC3101IRHBR, Y1 ABM3-12.000MHZ-D2Y-T

Commit message: routing...
Parts:
- added FID5: Fiducial, Fiducial:Fiducial_1.5mm_Mask3mm, B.Cu at (54.0, 152.5)
- added FID6: Fiducial, Fiducial:Fiducial_1.5mm_Mask3mm, B.Cu at (54.0, 27.0)
- added FID7: Fiducial, Fiducial:Fiducial_1.5mm_Mask3mm, B.Cu at (228.0, 152.5)
- added FID8: Fiducial, Fiducial:Fiducial_1.5mm_Mask3mm, B.Cu at (228.0, 27.0)
- moved C76 31.2 mm to (61.8, 33.2)
- moved C77 31.2 mm to (59.7, 33.2)
- moved U7 31.2 mm to (60.5, 37.0)
- moved J6 6.20 mm to (100.7, 47.0)
- moved J10 5.83 mm to (86.7, 48.6)
- moved R36 4.16 mm to (86.3, 109.3), turned to 180 degrees
Connections:
- C26 pad 1: +3.3VA -> /+3.3V_AUX2
- C27 pad 1: +3.3VA -> /+3.3V_AUX2
- C28 pad 1: +3.3VA -> /+3.3V_AUX2
- C29 pad 1: +3.3VA -> /+3.3V_AUX2
- C30 pad 1: +3.3VA -> /+3.3V_AUX2
- C36 pad 1: +3.3VA -> /+3.3V_AUX2
- C37 pad 1: +3.3VA -> /+3.3V_AUX2
- C38 pad 1: +3.3VA -> /+3.3V_AUX2
- C39 pad 1: +3.3VA -> /+3.3V_AUX2
- C40 pad 1: +3.3VA -> /+3.3V_AUX2
- C49 pad 1: +3.3VA -> /+3.3V_AUX2
- C50 pad 1: +3.3VA -> /+3.3V_AUX2
- C55 pad 1: +3.3VA -> /+3.3V_AUX1
- C56 pad 1: +3.3VA -> /+3.3V_AUX1
- C69 pad 1: +3.3VA -> /+3.3V_AUX1
- C70 pad 1: +3.3VA -> /+3.3V_AUX1
- C71 pad 1: +3.3VA -> /+3.3V_AUX1
- C75 pad 1: +3.3VA -> /+3.3V_AUX2
- R14 pad 2: +3.3VA -> +3.3V
- R30 pad 2: +3.3VA -> /+3.3V_AUX1
- U10 pad 6: +3.3VA -> /+3.3V_AUX2
- U11 pad 6: +3.3VA -> /+3.3V_AUX1
- U11 pad 8: +3.3VA -> /+3.3V_AUX1
- U17 pad 28: +3.3VA -> /+3.3V_AUX1
- U17 pad 3: +3.3VA -> /+3.3V_AUX1
- U8 pad 6: +3.3VA -> /+3.3V_AUX2
- U9 pad 18: +3.3VA -> /+3.3V_AUX2
- U9 pad 24: +3.3VA -> /+3.3V_AUX2
- U9 pad 25: +3.3VA -> /+3.3V_AUX2
- U9 pad 7: +3.3VA -> /+3.3V_AUX2
Routing:
- net Net-(J10-Pin_1): track 1.51 -> 49.6 mm, vias 0 -> 1
- net Net-(J10-Pin_2): track 1.53 -> 47.1 mm, vias 0 -> 1
- net Net-(J6-Pin_1): track 1.55 -> 40.9 mm
- net Net-(J6-Pin_2): track 1.95 -> 35.9 mm
- net /+3.3V_AUX2: track 4.81 -> 31.4 mm
- net +3.3VA: track 20.0 -> 10.9 mm
- net /BUTTON_Y: track 0.00 -> 6.50 mm
- net /BUTTON_X: track 0.00 -> 6.50 mm
- net /BUTTON_U: track 0.00 -> 6.50 mm
- net /BUTTON_START: track 0.00 -> 6.50 mm
- net /BUTTON_SELECT: track 0.00 -> 6.50 mm
- net /BUTTON_R: track 0.00 -> 6.50 mm
- net /BUTTON_L: track 0.00 -> 6.50 mm
- net /BUTTON_D: track 0.00 -> 6.50 mm
- net /BUTTON_B: track 0.00 -> 6.50 mm
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
Commit message: routing
Parts:
- added C78: 1uF, Capacitor_SMD:C_0603_1608Metric, B.Cu at (128.0, 100.0)
- added C79: 1uF, Capacitor_SMD:C_0603_1608Metric, B.Cu at (128.0, 102.5)
- added C80: 1uF, Capacitor_SMD:C_0603_1608Metric, B.Cu at (128.0, 105.0)
- added U19: TPS7A0533PDBV, Package_TO_SOT_SMD:SOT-23-5, B.Cu at (123.4, 101.1)
- moved C76 44.1 mm to (82.9, 71.9), turned to -90 degrees
- moved C77 43.5 mm to (82.9, 70.0), turned to 90 degrees
- moved U13 40.0 mm to (130.2, 38.5), turned to 0 degrees
- moved U7 39.0 mm to (79.1, 71.2), turned to -90 degrees
- moved J10 14.8 mm to (101.2, 51.8)
- moved J6 13.6 mm to (87.5, 50.6)
- moved R19 11.2 mm to (66.2, 40.6), turned to 0 degrees
- moved R20 9.13 mm to (62.9, 61.9), turned to -90 degrees
- moved R21 6.64 mm to (83.1, 42.2)
- moved R18 5.15 mm to (73.4, 49.8), turned to 180 degrees
- moved R22 5.15 mm to (94.5, 41.9)
- moved R5 4.71 mm to (57.9, 100.8), turned to 180 degrees
- moved R13 2.52 mm to (130.4, 59.9), turned to 180 degrees
- moved R26 1.60 mm to (133.6, 111.1)
- moved R25 1.51 mm to (132.0, 111.1)
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Connections:
- net /LEFT_LOM renamed /LEFT_LOM_C
- net /LEFT_LOP renamed /LEFT_LOP_C
- net /RIGHT_LOM renamed /RIGHT_LOM_C
- net /RIGHT_LOP renamed /RIGHT_LOP_C
- C40 pad 1: /+3.3V_AUX2 -> /+3.3V_AUX2_C
- C40 pad 2: GND -> GND_C
- C41 pad 1: GND -> GND_C
- C43 pad 1: GND -> GND_C
- C49 pad 1: /+3.3V_AUX2 -> /+3.3V_AUX2_C
- C49 pad 2: GND -> GND_C
- C50 pad 1: /+3.3V_AUX2 -> /+3.3V_AUX2_C
- C50 pad 2: GND -> GND_C
- C51 pad 1: GND -> GND_C
- C52 pad 1: GND -> GND_C
- C55 pad 1: /+3.3V_AUX1 -> +3V3
- C56 pad 1: /+3.3V_AUX1 -> +3V3
- C75 pad 1: /+3.3V_AUX2 -> /+3.3V_AUX2_C
- C75 pad 2: GND -> GND_C
- C76 pad 1: +3.3V -> +3.3V_C
- C76 pad 2: GND -> GND_C
- C77 pad 1: +3.3V -> +3.3V_C
- C77 pad 2: GND -> GND_C
- D5 pad 3: GND -> GND_C
- D6 pad 3: GND -> GND_C
- D7 pad 3: GND -> GND_C
- D9 pad 3: GND -> GND_C
- J2 pad 27: /+3.3V_AUX1 -> /+3.3V_AUX2
- J2 pad 4: /+3.3V_AUX1 -> /+3.3V_AUX2
- J3 pad 1: unconnected-(J3-Pad1) -> /I2C1_SCL_C
- J3 pad 12: unconnected-(J3-Pad12) -> +3.3V_C
- J3 pad 14: GND -> GND_C
- J3 pad 15: unconnected-(J3-Pad15) -> /I2C1_SCL_C
- J3 pad 16: unconnected-(J3-Pad16) -> /I2C1_SDA_C
- J3 pad 17: GND -> GND_C
- J3 pad 19: unconnected-(J3-Pad19) -> +3.3V_C
- J3 pad 2: GND -> GND_C
- J3 pad 23: +5V -> +5V_C
- J3 pad 27: unconnected-(J3-Pad27) -> /+3.3V_AUX2_C
- J3 pad 29: GND -> GND_C
- J3 pad 30: unconnected-(J3-Pad30) -> /I2C1_SDA_C
- J3 pad 4: unconnected-(J3-Pad4) -> /+3.3V_AUX2_C
- J3 pad 8: +5V -> +5V_C
- J4 pad 1: +3.3VA -> /+3.3V_AUX2
- J8 pad 27: /+3.3V_AUX1 -> /+3.3V_AUX2
- J8 pad 4: /+3.3V_AUX1 -> /+3.3V_AUX2
- J9 pad 1: unconnected-(J9-Pad1) -> /I2C1_SDA_C
- J9 pad 12: unconnected-(J9-Pad12) -> +3.3V_C
- J9 pad 14: GND -> GND_C
- J9 pad 15: /EYESPI_SCL -> /I2C1_SCL_C
- J9 pad 16: unconnected-(J9-Pad16) -> /I2C1_SCL_C
- J9 pad 17: GND -> GND_C
- J9 pad 19: unconnected-(J9-Pad19) -> +3.3V_C
- J9 pad 2: GND -> GND_C
- J9 pad 23: unconnected-(J9-Pad23) -> +5V_C
- J9 pad 27: unconnected-(J9-Pad27) -> /+3.3V_AUX2_C
- J9 pad 29: GND -> GND_C
- J9 pad 30: /EYESPI_SDA -> /I2C1_SDA_C
- J9 pad 4: unconnected-(J9-Pad4) -> /+3.3V_AUX2_C
- J9 pad 8: +5V -> +5V_C
- R12 pad 2: +3.3V -> +3.3V_C
- R13 pad 2: +3.3V -> +3.3V_C
- R15 pad 2: +3.3V -> +3.3V_C
- R16 pad 2: +3.3V -> +3.3V_C
- R17 pad 2: +3.3V -> +3.3V_C
- R18 pad 2: +3.3V -> +3.3V_C
- R19 pad 2: +3.3V -> +3.3V_C
- R20 pad 2: +3.3V -> +3.3V_C
- R21 pad 2: +3.3V -> +3.3V_C
- R22 pad 2: +3.3V -> +3.3V_C
- R30 pad 2: /+3.3V_AUX1 -> +3V3
- R40 pad 2: +3.3VA -> /+3.3V_AUX1
- SW10 pad 2: GND -> GND_C
- SW11 pad 2: GND -> GND_C
- SW2 pad 2: GND -> GND_C
- SW3 pad 2: GND -> GND_C
- SW4 pad 2: GND -> GND_C
- SW5 pad 2: GND -> GND_C
- SW6 pad 2: GND -> GND_C
- SW7 pad 2: GND -> GND_C
- SW8 pad 2: GND -> GND_C
- SW9 pad 2: GND -> GND_C
- U10 pad 1: +3.3VA -> GND_C
- U10 pad 6: /+3.3V_AUX2 -> /+3.3V_AUX2_C
- U10 pad 7: GND -> GND_C
- U11 pad 6: /+3.3V_AUX1 -> +3V3
- U11 pad 8: /+3.3V_AUX1 -> +3V3
- U16 pad S1: +3.3VA -> /+3.3V_CELL
- U18 pad 43: +3.3VA -> /+3.3V_CELL
- U7 pad 18: GND -> GND_C
- U7 pad 19: /EYESPI_SCL -> /I2C1_SCL_C
- U7 pad 20: /EYESPI_SDA -> /I2C1_SDA_C
- U7 pad 21: +3.3V -> +3.3V_C
- U7 pad 22: unconnected-(U7-~{INT}-Pad22) -> /INPUT_INT
- U7 pad 23: +3.3V -> +3.3V_C
- U7 pad 25: GND -> GND_C
- U7 pad 9: GND -> GND_C
- U8 pad 1: unconnected-(U8-~{SD}-Pad1) -> GND_C
- U8 pad 6: /+3.3V_AUX2 -> /+3.3V_AUX2_C
- U8 pad 7: GND -> GND_C
Routing:
- net /EYESPI_SDA: track 0.00 -> 180.5 mm, vias 0 -> 9
- net /EYESPI_SCL: track 0.00 -> 178.9 mm, vias 0 -> 11
- net +3.3V_C: track 0.00 -> 101.6 mm
- net /BUTTON_X: track 6.50 -> 70.7 mm
- net /I2C1_SCL_C: track 0.00 -> 54.9 mm, vias 0 -> 3
- net /BUTTON_A: track 6.50 -> 58.7 mm, vias 0 -> 1
- net /I2C1_SDA_C: track 0.00 -> 51.9 mm, vias 0 -> 3
- net /BUTTON_SELECT: track 6.50 -> 55.3 mm, vias 0 -> 1
- net /BUTTON_Y: track 6.50 -> 51.0 mm, vias 0 -> 1
- net Net-(U15-USB_DM): track 0.00 -> 43.2 mm, vias 0 -> 3
- net /BUTTON_START: track 6.50 -> 49.6 mm, vias 0 -> 1
- net Net-(U15-USB_DP): track 0.00 -> 40.8 mm, vias 0 -> 2
- net /BUTTON_B: track 6.50 -> 45.1 mm
- net /BUTTON_L: track 6.50 -> 40.1 mm, vias 0 -> 1
- net +3V3: track 32.9 -> 65.1 mm, vias 1 -> 6
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- added copper zone on F.Cu, net GND_C

Commit message: nearly done routing....
Parts:
- removed C78, C79, C80: 1uF, Capacitor_SMD:C_0603_1608Metric
- removed J12: Conn_Coaxial_Small, Connector_Coaxial:U.FL_Molex_MCRF_73412-0110_Vertical
- removed U16: 1042240820, 1042240820:1042240820_MOL
- removed U18: BG95M3LA-64-SGNS, Quectel_BG95M3LA:BG95_QWS
- removed U19: TPS7A0533PDBV, Package_TO_SOT_SMD:SOT-23-5
- added C81: 10uF, Capacitor_SMD:C_0805_2012Metric, F.Cu at (111.3, 110.7)
- C59, C60, C61, C62, C63, C64, C68: value 100n -> 100nF
- moved D5 22.4 mm to (100.0, 81.0)
- moved D7 22.1 mm to (78.0, 81.0), turned to 0 degrees
- moved C38 7.13 mm to (60.2, 126.0), turned to -90 degrees
- moved R14 1.90 mm to (105.7, 97.9)
- moved R44 1.70 mm to (112.5, 95.4)
- moved U13 1.70 mm to (131.6, 39.5)
- moved R45 1.40 mm to (111.0, 95.4)
- moved C42 1.08 mm to (57.2, 116.1), turned to 0 degrees
- moved C44 0.90 mm to (57.4, 113.8)
- moved C45 0.90 mm to (55.1, 113.4)
- moved C26 0.85 mm to (65.5, 113.4)
- moved D9 0.82 mm to (111.0, 81.0)
- moved C29 0.75 mm to (67.0, 113.4)
- moved C34 0.65 mm to (62.1, 113.4)
- moved C35 0.65 mm to (63.7, 113.4)
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Connections:
- C4 pad 1: +3V3 -> +3.3V
- C5 pad 1: +3V3 -> +3.3V
- C59 pad 1: +3V3 -> +3.3V
- C60 pad 1: +3V3 -> +3.3V
- C61 pad 1: +3V3 -> +3.3V
- C62 pad 1: +3V3 -> +3.3V
- C63 pad 1: +3V3 -> +3.3V
- C64 pad 1: +3V3 -> +3.3V
- C65 pad 1: +3V3 -> +3.3V
- C67 pad 1: +3V3 -> +3.3V
- C68 pad 1: +3V3 -> +3.3V
- D5 pad 1: +5V -> +5V_C
- D6 pad 1: +5V -> +5V_C
- D7 pad 1: +5V -> +5V_C
- D9 pad 1: +5V -> +5V_C
- J2 pad 20: unconnected-(J2-Pad20) -> /SPI1 MISO_C
- J2 pad 21: unconnected-(J2-Pad21) -> /SPI1 MOSI_C
- J2 pad 22: unconnected-(J2-Pad22) -> /SPI1 SCK_C
- J2 pad 5: unconnected-(J2-Pad5) -> /SPI1 MISO
- J2 pad 6: unconnected-(J2-Pad6) -> /SPI1 MOSI 
- J2 pad 7: unconnected-(J2-Pad7) -> /SPI1 SCK
- J3 pad 20: unconnected-(J3-Pad20) -> /SPI1 MISO_C
- J3 pad 21: unconnected-(J3-Pad21) -> /SPI1 MOSI_C
- J3 pad 22: unconnected-(J3-Pad22) -> /SPI1 SCK_C
- J3 pad 5: unconnected-(J3-Pad5) -> /SPI1 MISO_C
- J3 pad 6: unconnected-(J3-Pad6) -> /SPI1 MOSI_C
- J3 pad 7: unconnected-(J3-Pad7) -> /SPI1 SCK_C
- J8 pad 20: unconnected-(J8-Pad20) -> /SPI1 MISO
- J8 pad 21: unconnected-(J8-Pad21) -> /SPI1 MOSI 
- J8 pad 22: unconnected-(J8-Pad22) -> /SPI1 SCK
- J8 pad 5: unconnected-(J8-Pad5) -> /SPI1 MISO
- J8 pad 6: unconnected-(J8-Pad6) -> /SPI1 MOSI 
- J8 pad 7: unconnected-(J8-Pad7) -> /SPI1 SCK
- J9 pad 20: unconnected-(J9-Pad20) -> /SPI1 MISO_C
- J9 pad 21: unconnected-(J9-Pad21) -> /SPI1 MOSI_C
- J9 pad 22: unconnected-(J9-Pad22) -> /SPI1 SCK_C
- J9 pad 5: unconnected-(J9-Pad5) -> /SPI1 MISO_C
- J9 pad 6: unconnected-(J9-Pad6) -> /SPI1 MOSI _C
- J9 pad 7: unconnected-(J9-Pad7) -> /SPI1 SCK_C
- R36 pad 1: +3V3 -> +3.3V
- U1 pad 5: +3V3 -> +3.3V
- U14 pad 8: +3V3 -> +3.3V
- U15 pad 1: +3V3 -> +3.3V
- U15 pad 10: +3V3 -> +3.3V
- U15 pad 13: /BUTTON_R1 -> /SPI1 SCK
- U15 pad 14: /BUTTON_R2 -> /SPI1 MOSI 
- U15 pad 15: unconnected-(U15-GPIO12-Pad15) -> /SPI1 MISO
- U15 pad 16: unconnected-(U15-GPIO13-Pad16) -> /BUTTON_R1
- U15 pad 17: unconnected-(U15-GPIO14-Pad17) -> /BUTTON_R2
- U15 pad 22: +3V3 -> +3.3V
- U15 pad 33: +3V3 -> +3.3V
- U15 pad 42: +3V3 -> +3.3V
- U15 pad 43: +3V3 -> +3.3V
- U15 pad 44: +3V3 -> +3.3V
- U15 pad 48: +3V3 -> +3.3V
- U15 pad 49: +3V3 -> +3.3V
Routing:
- net +3.3V: track 12.2 -> 207.9 mm, vias 0 -> 12
- net +3.3V_C: track 101.6 -> 251.4 mm, vias 0 -> 8
- net /RESET: track 0.00 -> 120.6 mm, vias 0 -> 4
- net /+3.3V_AUX2: track 49.9 -> 169.1 mm, vias 2 -> 9
- net +5V_C: track 4.82 -> 117.1 mm, vias 0 -> 2
- net /+3.3V_AUX2_C: track 17.1 -> 121.6 mm, vias 0 -> 5
- net /I2S_RXD: track 0.00 -> 81.1 mm, vias 0 -> 2
- net /I2S_TXD: track 0.00 -> 72.3 mm, vias 0 -> 2
- net /I2S_LRCLK: track 0.00 -> 67.4 mm, vias 0 -> 2
- net /I2C1_SDA_C: track 51.9 -> 117.6 mm
- net /I2C1_SCL_C: track 54.9 -> 120.5 mm, vias 3 -> 4
- net /+3.3V_AUX1: track 20.1 -> 84.9 mm, vias 0 -> 3
- net +3V3: track 65.1 -> 8.17 mm, vias 6 -> 0
- net /BUTTON_L2: track 4.27 -> 54.2 mm, vias 0 -> 1
- net /BUTTON_L1: track 3.54 -> 46.1 mm, vias 0 -> 1
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- added copper zone on In1.Cu, net (none)
- added copper zone on B.Cu, net GND_C
Other:
- outline, holes or cut-outs redrawn

Commit message: routing...
Parts:
- moved C76 0.17 mm to (83.1, 71.9)
Connections:
- J2 pad 1: /EYESPI_SCL -> /EYESPI_SDA
- J2 pad 16: /EYESPI_SDA -> /EYESPI_SCL
- J2 pad 20: /SPI1 MISO_C -> unconnected-(J2-Pad20)
- J2 pad 21: /SPI1 MOSI_C -> unconnected-(J2-Pad21)
- J2 pad 22: /SPI1 SCK_C -> unconnected-(J2-Pad22)
- J2 pad 24: unconnected-(J2-Pad24) -> /SPI1 SCK
- J2 pad 25: unconnected-(J2-Pad25) -> /SPI1 MOSI
- J2 pad 26: unconnected-(J2-Pad26) -> /SPI1 MISO
- J2 pad 6: /SPI1 MOSI  -> /SPI1 MOSI
- J3 pad 1: /I2C1_SCL_C -> /I2C1_SDA_C
- J3 pad 16: /I2C1_SDA_C -> /I2C1_SCL_C
- J3 pad 20: /SPI1 MISO_C -> unconnected-(J3-Pad20)
- J3 pad 21: /SPI1 MOSI_C -> unconnected-(J3-Pad21)
- J3 pad 22: /SPI1 SCK_C -> unconnected-(J3-Pad22)
- J3 pad 24: unconnected-(J3-Pad24) -> /SPI1 SCK_C
- J3 pad 25: unconnected-(J3-Pad25) -> /SPI1 MOSI_C
- J3 pad 26: unconnected-(J3-Pad26) -> /SPI1 MISO_C
- J8 pad 20: /SPI1 MISO -> unconnected-(J8-Pad20)
- J8 pad 21: /SPI1 MOSI  -> unconnected-(J8-Pad21)
- J8 pad 22: /SPI1 SCK -> unconnected-(J8-Pad22)
- J8 pad 24: unconnected-(J8-Pad24) -> /SPI1 SCK
- J8 pad 25: unconnected-(J8-Pad25) -> /SPI1 MOSI
- J8 pad 26: unconnected-(J8-Pad26) -> /SPI1 MISO
- J8 pad 6: /SPI1 MOSI  -> /SPI1 MOSI
- J9 pad 20: /SPI1 MISO_C -> unconnected-(J9-Pad20)
- J9 pad 21: /SPI1 MOSI_C -> unconnected-(J9-Pad21)
- J9 pad 22: /SPI1 SCK_C -> unconnected-(J9-Pad22)
- J9 pad 24: unconnected-(J9-Pad24) -> /SPI1 SCK_C
- J9 pad 25: unconnected-(J9-Pad25) -> /SPI1 MOSI_C
- J9 pad 26: unconnected-(J9-Pad26) -> /SPI1 MISO_C
- U15 pad 14: /SPI1 MOSI  -> /SPI1 MOSI
Routing:
- net /SPI1 MOSI: track 0.00 -> 113.5 mm, vias 0 -> 4
- net /SPI1 SCK: track 2.39 -> 110.2 mm, vias 0 -> 4
- net /SPI1 MISO: track 2.38 -> 47.9 mm, vias 0 -> 3
- net +3.3V: track 207.9 -> 230.7 mm, vias 12 -> 14
- net /EYESPI_TSCS: track 0.00 -> 16.6 mm, vias 0 -> 2
- net /EYESPI_TFTCS: track 0.00 -> 16.6 mm, vias 0 -> 2
- net /EYESPI_SCL: track 190.2 -> 181.0 mm
- net /I2C1_SCL_C: track 120.5 -> 111.8 mm
- net /I2C1_SDA_C: track 117.6 -> 110.0 mm
- net /USB_VBUS: track 23.5 -> 29.5 mm, vias 6 -> 8
- net /RESET: track 120.6 -> 117.0 mm
- net /I2S_MCLK: track 31.1 -> 27.9 mm
- net /SPI1 MOSI : track 2.38 -> 0.00 mm
- net /I2S_BC: track 38.2 -> 35.9 mm
- net /I2S_LRCLK: track 67.4 -> 65.6 mm
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
Commit message: more routing
Parts:
- added R46: 100k, Resistor_SMD:R_0603_1608Metric, F.Cu at (86.5, 69.2)
- moved U13 3.63 mm to (130.4, 36.0)
- turned TH1 to -90 degrees
Connections:
- J2 pad 9: unconnected-(J2-Pad9) -> /INPUT_INT
- J3 pad 9: unconnected-(J3-Pad9) -> /INPUT_INT_C
- J8 pad 9: unconnected-(J8-Pad9) -> /INPUT_INT
- J9 pad 9: unconnected-(J9-Pad9) -> /INPUT_INT_C
- U13 pad 1: unconnected-(U13-VCC-Pad1) -> /+3.3V_AUX2_C
- U13 pad 2: unconnected-(U13-OUTPUT-Pad2) -> /LID_SENSE
- U13 pad 3: unconnected-(U13-GND-Pad3) -> GND_C
- U7 pad 12: unconnected-(U7-P1_2-Pad12) -> /LID_SENSE
- U7 pad 22: /INPUT_INT -> /INPUT_INT_C
- U7 pad 24: /RESET -> Net-(U7-~{RESET})
Routing:
- net /SPI1 MISO_C: track 0.00 -> 114.6 mm, vias 0 -> 5
- net /SPI1 SCK_C: track 0.00 -> 107.0 mm, vias 0 -> 4
- net /SPI1 MOSI_C: track 0.00 -> 103.3 mm, vias 0 -> 3
- net /SPI1 MISO: track 47.9 -> 122.9 mm, vias 3 -> 5
- net +5V: track 71.8 -> 136.2 mm, vias 3 -> 4
- net Net-(U2-TS): track 0.00 -> 20.5 mm, vias 0 -> 1
- net /SPI1 SCK: track 110.2 -> 121.2 mm, vias 4 -> 5
- net /I2C1_SCL_C: track 111.8 -> 122.0 mm, vias 4 -> 6
- net /I2C1_SDA_C: track 110.0 -> 119.9 mm, vias 3 -> 5
- net Net-(D5-DOUT): track 0.00 -> 8.11 mm, vias 0 -> 2
- net GND: track 1.49 -> 7.99 mm, vias 52 -> 171
- net /SPI1 MOSI: track 113.5 -> 119.4 mm, vias 4 -> 5
- net Net-(U3-EN): track 23.4 -> 26.8 mm, vias 6 -> 7
- net /+3.3V_AUX2: track 170.5 -> 173.7 mm
- net Net-(J5-3V3-Pad1): track 25.7 -> 23.9 mm
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- removed copper zone on In1.Cu, net (none)
Other:
- outline, holes or cut-outs redrawn
