File: PortaPi_R1/PortaPi_R1.kicad_pcb (KiCad board)
At the start: 4 copper layers, 184.2 x 131 mm, 199 parts, among them J1 USB_C_Receptacle, J10 SpeakerOut, J11 Conn_Coaxial_Small, J2 DF40HC3.0-30DS-0.4V51, J3 DF40HC3.0-30DP, J4 FPC 0.5mmP 18 Pin, J5 Raspberry_Pi_2_3, J6 SpeakerOut, J7 AudioJack4, J8 DF40HC3.0-30DS-0.4V51, J9 DF40HC3.0-30DP, SW1 SW_Slide_DPDT, SW10 SW_SPST, SW11 SW_SPST, SW12 BOOT, SW13 SW_SPST, SW14 SW_SPST, SW15 SW_SPST, SW16 SW_SPST, SW2 A, SW3 X, SW4 B, SW5 Y, SW6 L, SW7 R, SW8 U, SW9 D, U1 TPS7A0533PDBV, U10 PAM8302AAD, U11 BME680, U12 RAK3172, U13 SM351LT, U14 W25Q128JVS, U15 RP2040, U17 BNO055, U2 BQ24072RGT, U3 TPS61252DSG, U4 TPS7A0533PDBV, U5 LTC2942, U6 TPS7A0533PDBV, U7 PCAL6416AHF, U8 PAM8302AAD, U9 TLV320AIC3101IRHBR, Y1 ABM3-12.000MHZ-D2Y-T

Commit message: misc work
Parts:
- J2: value DF40HC3.0-30DS-0.4V51 -> DF40HC4.0-30DS-0.4V51
- moved R46 1.78 mm to (85.0, 70.2), turned to -90 degrees
Routing:
- net Net-(U7-~{RESET}): track 0.00 -> 5.79 mm
- net +3.3V_C: track 252.2 -> 253.6 mm
Changed lines of the file:
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@@
 			)
 		)
-		(property "Value" "DF40HC3.0-30DS-0.4V51"
+		(property "Value" "DF40HC4.0-30DS-0.4V51"
 			(at 0 0 -90)
 			(unlocked yes)
@@
 	(footprint "Resistor_SMD:R_0603_1608Metric"
 		(layer "F.Cu")
-		(at 86.525 69.25)
+		(at 85 70.175 -90)
 		(descr "Resistor SMD 0603 (1608 Metric), square (rectangular) end terminal, IPC_7351 nominal, (Body size source: IPC-SM-782 page 72, https://www.pcb-3d.com/wordpress/wp-content/uploads/ipc-sm-782a_amendment_1_and_2.pdf), generated with kicad-footprint-generator")
 		(tags "resistor")
 		(property "Reference" "R46"
-			(at 0 -1.43 360)
+			(at 0 -1.43 90)
 			(layer "F.SilkS")
 			(effects
@@
 		)
 		(property "Value" "100k"
-			(at 0 1.43 360)
+			(at 0 1.43 90)
 			(layer "F.Fab")
 			(effects
@@
 		)
 		(property "Footprint" "Resistor_SMD:R_0603_1608Metric"
-			(at 0 0 0)
+			(at 0 0 -90)
 			(unlocked yes)
 			(layer "F.Fab")
@@
 		)
 		(property "Datasheet" ""
-			(at 0 0 0)
+			(at 0 0 -90)
 			(unlocked yes)
 			(layer "F.Fab")
@@
 		)
 		(property "Description" "Resistor"
-			(at 0 0 0)
+			(at 0 0 -90)
 			(unlocked yes)
 			(layer "F.Fab")
@@
 		(attr smd)
 		(fp_line
-			(start -0.237258 -0.5225)
-			(end 0.237258 -0.5225)
+			(start -0.237258 0.5225)
+			(end 0.237258 0.5225)
 			(stroke
 				(width 0.12)
@@
 		)
 		(fp_line
-			(start -0.237258 0.5225)
-			(end 0.237258 0.5225)
+			(start -0.237258 -0.5225)
+			(end 0.237258 -0.5225)
 			(stroke
 				(width 0.12)
@@
 		)
 		(fp_line
-			(start -1.48 -0.73)
-			(end 1.48 -0.73)
+			(start -1.48 0.73)
+			(end -1.48 -0.73)
 			(stroke
 				(width 0.05)
@@
 		)
 		(fp_line
-			(start -1.48 0.73)
-			(end -1.48 -0.73)
+			(start 1.48 0.73)
+			(end -1.48 0.73)
 			(stroke
 				(width 0.05)
@@
 		)
 		(fp_line
-			(start 1.48 -0.73)
-			(end 1.48 0.73)
+			(start -1.48 -0.73)
+			(end 1.48 -0.73)
 			(stroke
 				(width 0.05)
@@
 		)
 		(fp_line
-			(start 1.48 0.73)
-			(end -1.48 0.73)
+			(start 1.48 -0.73)
+			(end 1.48 0.73)
 			(stroke
 				(width 0.05)
@@
 		)
 		(fp_line
-			(start -0.8 -0.4125)
-			(end 0.8 -0.4125)
+			(start -0.8 0.4125)
+			(end -0.8 -0.4125)
 			(stroke
 				(width 0.1)
@@
 		)
 		(fp_line
-			(start -0.8 0.4125)
-			(end -0.8 -0.4125)
+			(start 0.8 0.4125)
+			(end -0.8 0.4125)
 			(stroke
 				(width 0.1)
@@
 		)
 		(fp_line
-			(start 0.8 -0.4125)
-			(end 0.8 0.4125)
+			(start -0.8 -0.4125)
+			(end 0.8 -0.4125)
 			(stroke
 				(width 0.1)
@@
 		)
 		(fp_line
-			(start 0.8 0.4125)
-			(end -0.8 0.4125)
+			(start 0.8 -0.4125)
+			(end 0.8 0.4125)
 			(stroke
 				(width 0.1)
@@
 		)
 		(fp_text user "${REFERENCE}"
-			(at 0 0 360)
+			(at 0 0 90)
 			(layer "F.Fab")
 			(effects
@@
 		)
 		(pad "1" smd roundrect
-			(at -0.825 0)
+			(at -0.825 0 270)
 			(size 0.8 0.95)
 			(layers "F.Cu" "F.Paste" "F.Mask")
@@
 		)
 		(pad "2" smd roundrect
-			(at 0.825 0)
+			(at 0.825 0 270)
 			(size 0.8 0.95)
 			(layers "F.Cu" "F.Paste" "F.Mask")
@@
 	)
 	(via
-		(at 114.95 100.55)
+		(at 115.05 100.05)
 		(size 0.35)
 		(drill 0.2)
@@
 	)
 	(segment
-		(start 136.35 118.007866)
-		(end 136.35 110.75)
-		(width 0.762)
-		(layer "In2.Cu")
-		(net 45)
-	)
-	(segment
 		(start 97.339754 98.15)
 		(end 98.149354 97.3404)
@@
 	)
 	(segment
-		(start 107.480257 97.3404)
-		(end 98.149354 97.3404)
+		(start 133.85 108.25)
+		(end 131.75 108.25)
 		(width 0.762)
 		(layer "In2.Cu")
@@
 	)
 	(segment
-		(start 85.85 98.15)
-		(end 97.339754 98.15)
+		(start 131.75 108.25)
+		(end 122.3 98.8)
 		(width 0.762)
 		(layer "In2.Cu")
@@
 	)
 	(segment
-		(start 57.279864 113.240714)
-		(end 62.249541 113.240714)
+		(start 85.85 98.15)
+		(end 97.339754 98.15)
 		(width 0.762)
 		(layer "In2.Cu")
@@
 	)
 	(segment
-		(start 131.75 108.25)
-		(end 121.094 97.594)
+		(start 57.279864 113.240714)
+		(end 62.249541 113.240714)
 		(width 0.762)
 		(layer "In2.Cu")
@@
 	)
 	(segment
-		(start 62.501626 113.4928)
-		(end 66 113.4928)
+		(start 136.35 110.75)
+		(end 133.85 108.25)
 		(width 0.762)
 		(layer "In2.Cu")
@@
 	)
 	(segment
-		(start 135.907256 118.45061)
-		(end 136.35 118.007866)
+		(start 136.35 118.007866)
+		(end 136.35 110.75)
 		(width 0.762)
 		(layer "In2.Cu")
@@
 	)
 	(segment
-		(start 133.85 108.25)
-		(end 131.75 108.25)
+		(start 62.501626 113.4928)
+		(end 66 113.4928)
+		(width 0.762)
+		(layer "In2.Cu")
+		(net 45)
+	)
+	(segment
+		(start 135.907256 118.45061)
+		(end 136.35 118.007866)
 		(width 0.762)
 		(layer "In2.Cu")
@@
 	)
 	(segment
+		(start 108.939857 98.8)
+		(end 107.480257 97.3404)
+		(width 0.762)
+		(layer "In2.Cu")
+		(net 45)
+	)
+	(segment
 		(start 62.249541 113.240714)
 		(end 62.501626 113.4928)
@@
 	)
 	(segment
-		(start 121.094 97.594)
-		(end 107.733857 97.594)
-		(width 0.762)
-		(layer "In2.Cu")
-		(net 45)
-	)
-	(segment
 		(start 135.800607 118.557259)
 		(end 135.907256 118.45061)
@@
 	)
 	(segment
-		(start 136.35 110.75)
-		(end 133.85 108.25)
+		(start 122.3 98.8)
+		(end 108.939857 98.8)
 		(width 0.762)
 		(layer "In2.Cu")
@@
 	)
 	(segment
-		(start 107.733857 97.594)
-		(end 107.480257 97.3404)
+		(start 107.480257 97.3404)
+		(end 98.149354 97.3404)
 		(width 0.762)
 		(layer "In2.Cu")
@@
 	)
 	(segment
+		(start 84 71.05)
+		(end 84.95 71.05)
+		(width 0.1524)
+		(layer "F.Cu")
+		(net 108)
+	)
+	(segment
 		(start 72.800453 41.4)
 		(end 73.7 41.4)
@@
 	)
 	(segment
+		(start 84.95 71.05)
+		(end 85 71)
+		(width 0.1524)
+		(layer "F.Cu")
+		(net 108)
+	)
+	(segment
 		(start 84.875 42.225)
 		(end 94 42.225)
@@
 	)
 	(segment
+		(start 83.75 70.8)
+		(end 84 71.05)
+		(width 0.1524)
+		(layer "F.Cu")
+		(net 108)
+	)
+	(segment
 		(start 136.486791 58.400001)
 		(end 136.33559 58.2488)
@@
 		(net 256)
 	)
+	(segment
+		(start 81.05 68.5)
+		(end 81.05 69.9525)
+		(width 0.1524)
+		(layer "F.Cu")
+		(net 258)
+	)
+	(segment
+		(start 84.05 68.5)
+		(end 81.05 68.5)
+		(width 0.1524)
+		(layer "F.Cu")
+		(net 258)
+	)
+	(segment
+		(start 85 69.35)
+		(end 84.9 69.35)
+		(width 0.1524)
+		(layer "F.Cu")
+		(net 258)
+	)
+	(segment
+		(start 84.9 69.35)
+		(end 84.05 68.5)
+		(width 0.1524)
+		(layer "F.Cu")
+		(net 258)
+	)
+	(segment
+		(start 81.05 69.9525)
+		(end 81.0775 69.98)
+		(width 0.1524)
+		(layer "F.Cu")
+		(net 258)
+	)
 	(zone
